File: licheerv_nano_base/licheerv_nano_base.kicad_sch (KiCad schematic)
At the start: 112 parts, among them J1 USB STM32, J10 Valve, J11 ETH_IN, J12 ETH_OUT, J13 Compressor, J14 DebugUART, J15 Weight, J16 Malibotti, J17 Robot, J18 SWDBG, J19 IO, J2 Barrel_Jack_Switch, J3 TOF1, J4 TOF1, J5 TOF1, J6 TOF1, J7 STEP1, J8 STEP2, J9 Conveyor, Q1 BC807, Q2 IRLML6344, Q3 IRLML6344, Q4 IRLML6344, U1 TPS54202DDC, U2 STM32G431RBTx, U3 HX711, U5 TMC2209, U6 TMC2209

Commit message: Initial commit lichee_rv_nano_base pcb
Parts:
- added FID2: Fiducial, liebler_DRAWINGS:barrel_jack_positive_polarity, symbol Mechanical:Fiducial
- added R11: 10k, Resistor_SMD:R_0201_0603Metric, symbol Device:R
- added U4: DCDC_MP2315, liebler_MODULES:DCDC_MP2315, symbol liebler_MODULES:DCDC_MP2315
- C5, C7: footprint Capacitor_SMD:C_0603_1608Metric -> Capacitor_SMD:C_0805_2012Metric
- C8: value 1u -> 2u2
- J2: value Barrel_Jack_Switch -> DC IN
- J3: value TOF1 -> TOF3
- J4: value TOF1 -> TOF2
- L1: footprint liebler_PASSIVES:L_0630 -> Inductor_SMD:L_Abracon_ASPI-0630LR
- LS2: value Speaker_withoutTerminals -> Speaker
- Q1: footprint Package_TO_SOT_SMD:SOT-23_Handsoldering -> liebler_SEMICONDUCTORS:SOT-23_smaller
- R2: footprint Resistor_SMD:R_0201_0603Metric -> Resistor_SMD:R_0402_1005Metric
- R5, R6, R7: footprint Resistor_SMD:R_0805_2012Metric_Pad1.20x1.40mm_HandSolder -> Resistor_SMD:R_0402_1005Metric
- R8: value 20k -> 10k; footprint Resistor_SMD:R_0805_2012Metric_Pad1.20x1.40mm_HandSolder -> Resistor_SMD:R_0201_0603Metric
- TP1: value Stepper_UART -> StepperUART
- U7: value ~ -> PoE->24V
Connections:
- net +9V: now also U4.1 (OUT+)
- net 5-24V: now also U4.3 (IN+)
- net GND: now also U4.2 (GND)
- net INT_TOF1: now also J4.3 (Pin_3), U2.13 (PA1); no longer J3.3 (Pin_3), U2.62 (PB9)
- net INT_TOF2: now also J5.3 (Pin_3), U2.12 (PA0); no longer J4.3 (Pin_3), U2.13 (PA1)
- net INT_TOF3: now also J3.3 (Pin_3), U2.62 (PB9); no longer J5.3 (Pin_3), U2.12 (PA0)
- net MALIBOTTI_RXD: now also U8.27 (GPIOA18/U1T/P6); no longer U8.23 (GPIOA28/U2T)
- net MALIBOTTI_TXD: now also U8.28 (GPIOA19/U1R/P7); no longer U8.25 (GPIOA29/U2R)
- net ROBOT_RXD: now also U8.23 (GPIOA28/U2T); no longer U8.27 (GPIOA18/U1T/P6)
- net ROBOT_TXD: now also U8.25 (GPIOA29/U2R); no longer U8.28 (GPIOA19/U1R/P7)
- net i1c: now also J4.1 (Pin_1), U2.22 (PC4); no longer J3.1 (Pin_1), U2.51 (PA15)
- net i1d: now also J4.2 (Pin_2), U2.5 (PF0); no longer J3.2 (Pin_2), U2.60 (PB7)
- net i2c: now also J5.1 (Pin_1), U2.40 (PC8); no longer J4.1 (Pin_1), U2.22 (PC4)
- net i2d: now also J5.2 (Pin_2), U2.41 (PC9); no longer J4.2 (Pin_2), U2.5 (PF0)
- net i3c: now also J3.1 (Pin_1), U2.51 (PA15); no longer J5.1 (Pin_1), U2.40 (PC8)
- net i3d: now also J3.2 (Pin_2), U2.60 (PB7); no longer J5.2 (Pin_2), U2.41 (PC9)
- net at R7.1, U3.4 (VFB): now also R11.2; no longer R8.2
- net RX: now reaches J14.2 (Pin_2), U8.1 (GPIOA17/U0R/P5)
- net TX: now reaches J14.3 (Pin_3), U8.2 (GPIOA16/U0T/P4)
- new net: R11.1, R8.2
Other:
- note added: "Connectors"
- note added: "LicheeRV nano"
- note added: "Mech"
- note added: "PoE->24V"
- note added: "PoE-Splitter"
- note added: "Pullups"
- note added: "STM32"
- note added: "Stepper Various"
- note removed: "Stepper1_Step"
- note removed: "Stepper2_Step"
- moved on the sheet: C1, C10, C11, C12, C13, C14, C15, C16, C17, C18, C19, C2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

Commit message: lichee_rv_nano aka radxa zero 3e as ordered @ jlcpcb
Parts:
- removed C1, C29, C30, C42, C43: u1/35V, Capacitor_SMD:C_0603_1608Metric, symbol Device:C
- removed C10, C22: 10u, Capacitor_SMD:C_0805_2012Metric_Pad1.18x1.45mm_HandSolder, symbol Device:C
- removed C11, C13, C20, C21, C25, C26, C27, C28, C6: u1, Capacitor_SMD:C_0201_0603Metric, symbol Device:C
- removed C2: 10u/35V, Capacitor_SMD:C_0805_2012Metric, symbol Device:C
- removed C23, C24: 100uF, Capacitor_THT:CP_Radial_D6.3mm_P2.50mm, symbol Device:C_Polarized
- removed C3: u1/16V, Capacitor_SMD:C_0603_1608Metric, symbol Device:C
- removed C33, C35: 2u2, Capacitor_SMD:C_0402_1005Metric, symbol Device:C
- removed C34, C36: 22n/50V, Capacitor_SMD:C_0402_1005Metric, symbol Device:C
- removed C37, C38, C39, C40: 22u/35V, Capacitor_SMD:C_0805_2012Metric, symbol Device:C
- removed C4: 56p, Capacitor_SMD:C_0402_1005Metric, symbol Device:C
- removed C5, C7: 22u, Capacitor_SMD:C_0805_2012Metric, symbol Device:C
- removed D1: Motor, liebler_OPTO:LED_1206_3216Metric_ReverseMount, symbol Device:LED
- removed D2: Valve, liebler_OPTO:LED_1206_3216Metric_ReverseMount, symbol Device:LED
- removed D3: Compressor, liebler_OPTO:LED_1206_3216Metric_ReverseMount, symbol Device:LED
- removed H5, H7: MountingHole, MountingHole:MountingHole_3.2mm_M3, symbol Mechanical:MountingHole
- removed J1: USB STM32, liebler_CONN:USB_C_Receptacle_HRO_TYPE-C-31-M-12_smaller, symbol Connector:USB_C_Receptacle_USB2.0_16P
- removed J10: Valve, liebler_CONN:PhoenixContact_MC_1,5_2-G-3.5_1x02_P3.50mm_Horizontal_smallerCourtyard, symbol Connector_Generic:Conn_01x02
- removed J11: ETH_IN, liebler_CONN:RJ45_WithoutMagneticsTHT, symbol Connector:8P8C_Shielded
- removed J12: ETH_OUT, liebler_CONN:RJ45_WithoutMagneticsTHT, symbol Connector:8P8C_Shielded
- removed J13: Compressor, liebler_CONN:PhoenixContact_MC_1,5_2-G-3.5_1x02_P3.50mm_Horizontal_smallerCourtyard, symbol Connector_Generic:Conn_01x02
- removed J15: Weight, liebler_CONN:JST_XH_S4B-XH-A-1_1x04_P2.50mm_Horizontal_SmallerCourtyard, symbol Connector_Generic:Conn_01x04
- removed J18: SWDBG, liebler_CONN:PinHeader_1x03_P2.54mm_Vertical_smallerCourtyard, symbol Connector_Generic:Conn_01x03
- removed J2: DC IN, Connector_BarrelJack:BarrelJack_Horizontal, symbol Connector:Barrel_Jack_Switch
- removed J7: STEP1, liebler_CONN:JST_XH_S4B-XH-A-1_1x04_P2.50mm_Horizontal_SmallerCourtyard, symbol Connector_Generic:Conn_01x04
- removed J8: STEP2, liebler_CONN:JST_XH_S4B-XH-A-1_1x04_P2.50mm_Horizontal_SmallerCourtyard, symbol Connector_Generic:Conn_01x04
- removed J9: Conveyor, liebler_CONN:PhoenixContact_MC_1,5_2-G-3.5_1x02_P3.50mm_Horizontal_smallerCourtyard, symbol Connector_Generic:Conn_01x02
- removed L1: 10uH, Inductor_SMD:L_Abracon_ASPI-0630LR, symbol Device:L
- removed L2: 3u3, Inductor_SMD:L_0805_2012Metric_Pad1.15x1.40mm_HandSolder, symbol Device:L
- removed LS1: Speaker, TestPoint:TestPoint_2Pads_Pitch2.54mm_Drill0.8mm, symbol Device:Speaker
- removed LS2: Speaker, liebler_MECH:SPEAKER_2415, symbol liebler_MECH:Speaker_withoutTerminals
- removed NT1: NetTie_2, NetTie:NetTie-2_SMD_Pad0.5mm, symbol Device:NetTie_2
- removed Q1: BC807, liebler_SEMICONDUCTORS:SOT-23_smaller, symbol Transistor_BJT:BC807
- removed Q2, Q3, Q4: IRLML6344, Package_TO_SOT_SMD:SOT-23, symbol Transistor_FET:IRLML0030
- removed R1, R19, R20, R22, R23, R25, R26: 1k, Resistor_SMD:R_0402_1005Metric, symbol Device:R
- removed R10, R11, R21, R24, R27, R3, R8, R9: 10k, Resistor_SMD:R_0201_0603Metric, symbol Device:R
- removed R15, R16, R17, R18: r1, Resistor_SMD:R_1206_3216Metric, symbol Device:R
- removed R2: M1, Resistor_SMD:R_0402_1005Metric, symbol Device:R
- removed R4: 3k3, Resistor_SMD:R_0402_1005Metric, symbol Device:R
- removed R5, R6: k1, Resistor_SMD:R_0402_1005Metric, symbol Device:R
- removed R7: 8k2, Resistor_SMD:R_0402_1005Metric, symbol Device:R
- removed TP1: StepperUART, TestPoint:TestPoint_THTPad_1.0x1.0mm_Drill0.5mm, symbol Connector:TestPoint
- removed U1: TPS54202DDC, Package_TO_SOT_SMD:SOT-23-6_Handsoldering, symbol Regulator_Switching:TPS54202DDC
- removed U3: HX711, Package_SO:SOIC-16_3.9x9.9mm_P1.27mm, symbol Analog_ADC:HX711
- removed U4: DCDC_MP2315, liebler_MODULES:DCDC_MP2315, symbol liebler_MODULES:DCDC_MP2315
- removed U5, U6: TMC2209, Package_DFN_QFN:QFN-28-1EP_5x5mm_P0.5mm_EP3.75x3.75mm_ThermalVias, symbol liebler_SEMICONDUCTORS:TMC2209
- removed U7: PoE->24V, liebler_MODULES:XC7010_DCDC_ISOLATED_MODUEL, symbol liebler_MODULES:XC7010_MODULE
- removed U8: ~, liebler_MODULES:LicheeRV_Nano, symbol liebler_MODULES:LICHEE_RV_NANO
- added D4: Info, liebler_OPTO:LED_1206_3216Metric_ReverseMount, symbol Device:LED
- added J18: STLINK_V3_MINIE, Connector_IDC:IDC-Header_2x05_P2.54mm_Vertical, symbol Connector_Generic:Conn_02x05_Odd_Even
- added J21: STDC14, liebler_CONN:IDC_2x07_P1.27mm_Vertical, symbol Connector:Conn_ST_STDC14
- added J22: USB STM32, liebler_CONN:USB_C_Receptacle_HRO_TYPE-C-31-M-12_smaller, symbol Connector:USB_C_Receptacle_USB2.0_16P
- added J23, J24: IO, Connector_JST:JST_XH_B6B-XH-A_1x06_P2.50mm_Vertical, symbol Connector_Generic:Conn_01x06
- added R13, R28: 5k1, Resistor_SMD:R_0201_0603Metric, symbol Device:R
- added R29, R30: 10k, Resistor_SMD:R_0201_0603Metric, symbol Device:R
- added R31: 1k, Resistor_SMD:R_0402_1005Metric, symbol Device:R
- added X1: Radxa Zero 3E, liebler_MODULES:Radxa Zero 3E, symbol liebler_MODULES:Radxa_Zero_3E
- R12, R14: now not fitted; now left out of the parts list
Connections:
- net +3V3: now also J18.10 (Pin_10), J21.3 (VCC), R31.2, X1.1 (3V3), X1.17 (3V3)
- net +5V: now also X1.2 (5V), X1.4 (5V)
- net Compressor_PWM: now also X1.24 (G4C6/S3_CS0/PWM13/U9R/I3S_SDI)
- net Conveyor_PWM: now also X1.7 (G3C4/-/-/PWM14_M0)
- net GND: now also J18.2 (Pin_2), J21.11 (GNDDetect), J21.5 (GND), J21.7 (GND), J22.A1 (GND), J22.A12 (GND), J22.B1 (GND), J22.B12 (GND), J22.S1 (SHIELD), R13.2, R28.2, R30.1, X1.14 (GND), X1.20 (GND), X1.25 (GND), X1.30 (GND), X1.34 (GND), X1.39 (GND), X1.6 (GND), X1.9 (GND)
- net INT_RGB: now also X1.15 (G3B0)
- net INT_TOF3: now also U2.2 (PC13); no longer U2.62 (PB9)
- net IO1: now also U2.62 (PB9); no longer U2.58 (PB5)
- net IO2: now also U2.58 (PB5); no longer U2.56 (PB3)
- net MALIBOTTI_RXD: now also X1.5 (G1A1/U3T/PU!)
- net MALIBOTTI_TXD: now also X1.3 (G1A0/U3R/PU!)
- net PB12: now also D4.1 (K), J23.1 (Pin_1)
- net PB13: now also J23.2 (Pin_2)
- net ROBOT_RXD: now also X1.18 (G3B2/U4T/PWM9)
- net ROBOT_TXD: now also X1.16 (G3B1/U4R/PWM8)
- net RX: now also X1.8 (U2T)
- net SCL: now also X1.28 (G4B3/-/-/I4C_SCL/I2S_SDO/PU!)
- net SDA: now also X1.27 (G4B2/-/I2S_SDI/I4C_SDA/PU!)
- net SPI1_MISO: now also X1.21 (G4C5/S3_MISO/I3S_SDO/PWM12/U9T)
- net SPI1_MOSI: now also X1.19 (G4C3/S3MOSI/I3S_SCLK/PWM15)
- net SPI1_NSS: now also X1.22 (G3C1/-/-/-/I1S_SDO2)
- net SPI1_SCK: now also X1.23 (G4C2/S3_CLK/I3S_MCLK/PWM14)
- net STM32BOOT_RXD: now also J18.4 (Pin_4), J21.13 (VCP_RX), X1.32 (G3C2/U5T/-/-/I2S_SDO3)
- net STM32BOOT_TXD: now also J18.6 (Pin_6), J21.14 (VCP_TX), X1.33 (G3C3/-/I1S_SCLK/-/U5R)
- net STM32_BOOT: now also X1.12 (G3A3)
- net STM32_RESET: now also J18.8 (Pin_8), J21.12 (~{RST}), X1.13 (G3A2/-/-/I2S3_MCLK)
- net SWCLK: now also J18.7 (Pin_7), J21.6 (JCLK/SWCLK)
- net SWDIO: now also J18.5 (Pin_5), J21.4 (JTMS/SWDIO)
- net T15C1: now also J23.3 (Pin_3)
- net T15C2: now also J23.4 (Pin_4)
- net T1C1-LU1R: now also J24.4 (Pin_4)
- net T1C2-LU1T: now also J24.3 (Pin_3)
- net T1C3: now also J24.2 (Pin_2)
- net T1C4: now also J24.1 (Pin_1)
- net T8C1: now also J23.5 (Pin_5)
- net T8C2: now also J23.6 (Pin_6)
- net TX: now also X1.10 (U2R)
- net USBPD_D+: now also J22.A6 (D+), J22.B6 (D+)
- net USBPD_D-: now also J22.A7 (D-), J22.B7 (D-)
- net Valve: now also X1.36 (G3A7)
- net PC14: now reaches U2.3 (PC14)
- net PC14: now also J24.6 (Pin_6)
- net PC15: now reaches U2.4 (PC15)
- net PC15: now also J24.5 (Pin_5)
- net USB_VSENSE: now reaches U2.6 (PF1)
- net USB_VSENSE: now also R29.1, R30.2
- net STEPPER_UART renamed U3R
- new net: J22.A5 (CC1), R13.1
- new net: J22.B5 (CC2), R28.1
- new net: D4.2 (A), R31.1
- new net +5VP: J22.A4 (VBUS), J22.A9 (VBUS), J22.B4 (VBUS), J22.B9 (VBUS), R29.2
- new net SWO: J18.9 (Pin_9), J21.8 (JTDO/SWO), U2.56 (PB3)
- no-connect marks 21 -> 13
Other:
- added sheet actors (actors.kicad_sch)
- added sheet psu (psu.kicad_sch)
- added sheet sensors (sensors.kicad_sch)
- note added: "Radxa Zero 3E"
- note added: "STM32 Debug"
- note added: "USB Data"
- note removed: "Barrel Jack 24V"
- note removed: "Compressor"
- note removed: "Compressor_PWM"
- note removed: "Conveyor"
- note removed: "Conveyor_PWM"
- note removed: "LicheeRV nano"
- note removed: "PSU"
- note removed: "PoE->24V"
- note removed: "PoE-Splitter"
- note removed: "Stepper Driver 1"
- note removed: "Stepper Driver 2"
- note removed: "Stepper Various"
- note removed: "USB PD"
- note removed: "Valve"
- note removed: "Weight Cell DAC"
- moved on the sheet: C12, C14, C15, C16, C17, C18, C19, C8, C9, FB1, FID2, H1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
