File: radxa_zero_3e_control_unit/actors.kicad_sch (KiCad schematic)
At the start: 51 parts, among them J10 Valve, J13 Compressor, J20 Bus-Servo, J7 STEP1, J8 STEP2, J9 Conveyor, Q2 IRLML6344, Q3 IRLML6344, Q4 IRLML6344, U5 TMC2209, U6 TMC2209

Commit message: Various
Parts:
- C23: footprint Capacitor_THT:CP_Radial_D6.3mm_P2.50mm -> Capacitor_THT:CP_Radial_D8.0mm_P2.50mm
Connections:
- net +3V3: now also U5.9 (MS1_AD0)
- net GND: no longer U5.9 (MS1_AD0)
Changed lines of the file:
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@@
 	(symbol
 		(lib_id "power:GND")
-		(at 35.56 38.1 270)
+		(at 35.56 121.92 270)
 		(unit 1)
 		(exclude_from_sim no)
@@
 		(fields_autoplaced yes)
 		(property "Reference" "#PWR049"
-			(at 29.21 38.1 0)
+			(at 29.21 121.92 0)
 			(effects
 				(font
@@
 		)
 		(property "Value" "GND"
-			(at 31.75 38.0999 90)
+			(at 31.75 121.9199 90)
 			(effects
 				(font
@@
 		)
 		(property "Footprint" ""
-			(at 35.56 38.1 0)
+			(at 35.56 121.92 0)
 			(effects
 				(font
@@
 		)
 		(property "Datasheet" ""
-			(at 35.56 38.1 0)
+			(at 35.56 121.92 0)
 			(effects
 				(font
@@
 		)
 		(property "Description" "Power symbol creates a global label with name \"GND\" , ground"
-			(at 35.56 38.1 0)
+			(at 35.56 121.92 0)
 			(effects
 				(font
@@
 	)
 	(symbol
+		(lib_id "power:+3V3")
+		(at 35.56 38.1 90)
+		(unit 1)
+		(exclude_from_sim no)
+		(in_bom yes)
+		(on_board yes)
+		(dnp no)
+		(fields_autoplaced yes)
+		(property "Reference" "#PWR0115"
+			(at 39.37 38.1 0)
+			(effects
+				(font
+					(size 1.27 1.27)
+				)
+				(hide yes)
+			)
+		)
+		(property "Value" "+3V3"
+			(at 31.75 38.0999 90)
+			(effects
+				(font
+					(size 1.27 1.27)
+				)
+				(justify left)
+			)
+		)
+		(property "Footprint" ""
+			(at 35.56 38.1 0)
+			(effects
+				(font
+					(size 1.27 1.27)
+				)
+				(hide yes)
+			)
+		)
+		(property "Datasheet" ""
+			(at 35.56 38.1 0)
+			(effects
+				(font
+					(size 1.27 1.27)
+				)
+				(hide yes)
+			)
+		)
+		(property "Description" "Power symbol creates a global label with name \"+3V3\""
+			(at 35.56 38.1 0)
+			(effects
+				(font
+					(size 1.27 1.27)
+				)
+				(hide yes)
+			)
+		)
+		(pin "1"
+		)
+		(instances
+			(project "radxa_zero_3e_control_unit"
+				(path "/8d672852-c950-41bc-8e5f-2837fc931963/607480ec-6159-45fb-845c-991fd3ee49c5"
+					(reference "#PWR0115")
+					(unit 1)
+				)
+			)
+		)
+	)
+	(symbol
 		(lib_name "IRLML0030_1")
 		(lib_id "Transistor_FET:IRLML0030")
@@
 			)
 		)
-		(property "Footprint" "Capacitor_THT:CP_Radial_D6.3mm_P2.50mm"
+		(property "Footprint" "Capacitor_THT:CP_Radial_D8.0mm_P2.50mm"
 			(at 140.6652 39.37 0)
 			(effects
@@
 					(unit 1)
 				)
-			)
-		)
-	)
-	(symbol
-		(lib_id "power:GND")
-		(at 35.56 121.92 270)
-		(unit 1)
-		(exclude_from_sim no)
-		(in_bom yes)
-		(on_board yes)
-		(dnp no)
-		(fields_autoplaced yes)
-		(property "Reference" "#PWR053"
-			(at 29.21 121.92 0)
-			(effects
-				(font
-					(size 1.27 1.27)
-				)
-				(hide yes)
-			)
-		)
-		(property "Value" "GND"
-			(at 31.75 121.9199 90)
-			(effects
-				(font
-					(size 1.27 1.27)
-				)
-				(justify right)
-			)
-		)
-		(property "Footprint" ""
-			(at 35.56 121.92 0)
-			(effects
-				(font
-					(size 1.27 1.27)
-				)
-				(hide yes)
-			)
-		)
-		(property "Datasheet" ""
-			(at 35.56 121.92 0)
-			(effects
-				(font
-					(size 1.27 1.27)
-				)
-				(hide yes)
-			)
-		)
-		(property "Description" "Power symbol creates a global label with name \"GND\" , ground"
-			(at 35.56 121.92 0)
-			(effects
-				(font
-					(size 1.27 1.27)
-				)
-				(hide yes)
-			)
-		)
-		(pin "1"
-		)
-		(instances
-			(project "licheerv_nano_base"
-				(path "/8d672852-c950-41bc-8e5f-2837fc931963/607480ec-6159-45fb-845c-991fd3ee49c5"
-					(reference "#PWR053")
-					(unit 1)
-				)

Commit message: WIP, before repinning SUM32G431
Parts:
- J20: footprint Connector_Molex:Molex_SPOX_5267-03A_1x03_P2.50mm_Vertical -> Connector_Molex:Molex_SPOX_5268-03A_1x03_P2.50mm_Horizontal
Changed lines of the file:
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@@
 			)
 		)
-		(property "Footprint" "Connector_Molex:Molex_SPOX_5267-03A_1x03_P2.50mm_Vertical"
+		(property "Footprint" "Connector_Molex:Molex_SPOX_5268-03A_1x03_P2.50mm_Horizontal"
 			(at 213.36 97.79 0)
 			(effects

Commit message: Udated control unit pcb
Parts:
- C24: footprint Capacitor_THT:CP_Radial_D6.3mm_P2.50mm -> Capacitor_THT:CP_Radial_D8.0mm_P2.50mm
- C27, C28: footprint Capacitor_SMD:C_0201_0603Metric -> Capacitor_SMD:C_0402_1005Metric
- J20: footprint Connector_Molex:Molex_SPOX_5268-03A_1x03_P2.50mm_Horizontal -> Connector_Molex:Molex_SPOX_5267-03A_1x03_P2.50mm_Vertical
- J7, J8: footprint liebler_CONN:JST_XH_S4B-XH-A-1_1x04_P2.50mm_Horizontal_SmallerCourtyard -> liebler_CONN:JST_XH_B4B-XH-A_1x04_P2.50mm_Vertical_smaller
- R10, R21, R24, R27, R9: footprint Resistor_SMD:R_0201_0603Metric -> Resistor_SMD:R_0402_1005Metric
- R76, R77: footprint Resistor_SMD:R_0805_2012Metric_Pad1.20x1.40mm_HandSolder -> Resistor_SMD:R_0402_1005Metric
- TP1: footprint TestPoint:TestPoint_THTPad_1.0x1.0mm_Drill0.5mm -> TestPoint:TestPoint_THTPad_D1.0mm_Drill0.5mm
Connections:
- net +3V3: now also U5.10 (MS2_AD1); no longer U5.9 (MS1_AD0)
- net 5-24V: no longer J10.1 (Pin_1), J13.1 (Pin_1), J9.1 (Pin_1)
- net GND: now also U5.9 (MS1_AD0); no longer U5.10 (MS2_AD1)
- net Compressor_PWM renamed COMPRESSOR_T2C1
- net Conveyor_PWM renamed CONVEYOR_T2C2
- net ROBOT_RXD renamed ROBOT_U4T
- net ROBOT_TXD renamed ROBOT_U4R
- net Stepper1_Dir renamed STEPPER1_DIR
- net Stepper1_Step renamed STEPPER1_STEP
- net Stepper2_Dir renamed STEPPER2_DIR_T3C1_T8C1
- net Stepper2_Step renamed STEPPER2_STEP_T3C2_T8C2
- net Valve renamed VALVE
- new net +24V: J10.1 (Pin_1), J13.1 (Pin_1), J9.1 (Pin_1)
