File: pcb_control_unit_ethernet/pcb_control_unit_ethernet.kicad_pcb (KiCad board)
At the start: 2 copper layers, 188 x 65 mm, 179 parts, among them J1 STDC14, J10 TOF1, J11 RGB, J12 LightBarrier1, J13 LightBarrier2, J14 LightBarrier3, J15 PressureTransducer, J16 CAN, J17 STEP1, J18 STEP2, J19 Conveyor, J2 Micro_SD_Card_Det1, J20 Valve, J21 Bus-Servo, J22 Compressor, J23 Weight, J3 HR911105A, J4 DC IN, J5 USB STM32, J6 USB STM32, J7 Malibotti, J8 TOF3, J9 TOF2, Q1 IRLML6344, Q2 IRLML6344, Q3 IRLML6344, Q4 BC807, SW1 Reset, SW2 Boot, U1 STM32H563VITx, U10 SIT3051TK, U2 LAN8742A, U3 DCDC_MP2315, U4 TPS54202DDC, U5 AMS1117-3.3, U6 INA226, U7 TMC2209, U8 TMC2209, U9 HX711, X1 MT3608

Commit message: First time zero errors, but bad layout
Parts:
- added Y1: 25MHz, Crystal:Crystal_SMD_2016-4Pin_2.0x1.6mm, F.Cu at (129.3, 71.2)
- C35: footprint Capacitor_SMD:C_0402_1005Metric -> Capacitor_SMD:C_0201_0603Metric
- C52, C53: footprint Capacitor_THT:CP_Radial_D8.0mm_P2.50mm -> Capacitor_SMD:CP_Elec_6.3x7.7
- J11, J12, J13, J14, J15, J20, J22, J23, X1: moved to B.Cu
- R44, R46, R63: footprint Resistor_SMD:R_0402_1005Metric -> Resistor_SMD:R_0201_0603Metric
- moved R42 240.2 mm to (141.4, 120.0), turned to -90 degrees
- moved R40 235.7 mm to (136.2, 120.0), turned to -90 degrees
- moved R44 233.3 mm to (139.0, 101.5), turned to -90 degrees
- moved C49 231.8 mm to (132.8, 111.5)
- moved C37 231.5 mm to (144.1, 108.8), turned to 180 degrees
- moved J11 228.3 mm to (172.8, 61.5)
- moved R27 228.2 mm to (139.1, 73.1)
- moved R41 228.0 mm to (128.8, 119.9), turned to -90 degrees
- moved R28 226.2 mm to (137.3, 73.6), turned to -90 degrees
- moved C26 226.1 mm to (139.8, 79.7), turned to -90 degrees
- moved C47 225.5 mm to (142.7, 110.7), turned to 90 degrees
- moved C25 224.5 mm to (141.2, 72.2), turned to 90 degrees
- moved R39 223.9 mm to (123.9, 119.9), turned to -90 degrees
- moved R29 222.7 mm to (135.2, 65.0)
- moved C46 222.7 mm to (139.9, 107.2), turned to 180 degrees
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Connections:
- net Net-(U2-VDD1A) renamed /eth/ETH_VA
- C58 pad 1: +3.3VA -> /sensors/VA_HX711
- C60 pad 1: +3.3VA -> /sensors/VA_HX711
- J12 pad 1: LightBarrier1 -> Net-(J12-Pin_1)
- J12 pad 2: Net-(J12-Pin_2) -> GND
- J12 pad 3: GND -> LightBarrier1
- J13 pad 1: LightBarrier2 -> Net-(J13-Pin_1)
- J13 pad 2: Net-(J13-Pin_2) -> GND
- J13 pad 3: GND -> LightBarrier2
- J14 pad 1: LightBarrier3 -> Net-(J14-Pin_1)
- J14 pad 2: Net-(J14-Pin_2) -> GND
- J14 pad 3: GND -> LightBarrier3
- J15 pad 1: Net-(J15-Pin_1) -> +5V
- J15 pad 2: +5V -> GND
- J15 pad 3: GND -> Net-(J15-Pin_3)
- J21 pad 1: ROBOT_U4R -> ROBOT_RX
- J5 pad A5: USBPD_CC1 -> USBPD_CC2
- J5 pad B5: USBPD_CC2 -> USBPD_CC1
- J7 pad 1: MALIBOTTI_U1R -> MALIBOTTI_RX
- J7 pad 2: MALIBOTTI_U1T -> MALIBOTTI_TX
- JP1 pad 2: Net-(J13-Pin_2) -> Net-(J13-Pin_1)
- JP2 pad 2: Net-(J12-Pin_2) -> Net-(J12-Pin_1)
- JP3 pad 2: Net-(J14-Pin_2) -> Net-(J14-Pin_1)
- NT3 pad 2: +3.3VA -> /sensors/VA_HX711
- Q4 pad 2: +3.3VA -> /sensors/VA_HX711
- R29 pad 1: /eth/LED2 -> /eth/LED1
- R30 pad 1: /eth/LED1 -> /eth/LED2
- R37 pad 2: Net-(J15-Pin_1) -> Net-(J15-Pin_3)
- R43 pad 1: U3T -> STEPPER_TX
- R43 pad 2: STEPPER_UART -> STEPPER_RX
- R45 pad 2: CONVEYOR_T2C2 -> CONVEYOR_PWM
- R46 pad 2: STEPPER_UART -> STEPPER_RX
- R47 pad 2: CONVEYOR_T2C2 -> CONVEYOR_PWM
- R52 pad 1: ROBOT_U4T -> ROBOT_TX
- R52 pad 2: ROBOT_U4R -> ROBOT_RX
- R53 pad 2: COMPRESSOR_T2C1 -> COMPRESSOR_PWM
- R54 pad 2: ROBOT_U4R -> ROBOT_RX
- R55 pad 2: COMPRESSOR_T2C1 -> COMPRESSOR_PWM
- TP1 pad 1: STEPPER_UART -> STEPPER_RX
- U1 pad 1: U8T -> MALIBOTTI_TX
- U1 pad 15: PC0 -> USB_VSENSE
- U1 pad 23: T5C1 -> ETH_RST
- U1 pad 35: T3C3 -> PRESSURE_ADC
- U1 pad 38: U7R -> ROBOT_RX
- U1 pad 39: U7T -> ROBOT_TX
- U1 pad 58: U4R -> STEPPER_RX
- U1 pad 63: T3C1 -> CONVEYOR_PWM
- U1 pad 64: T8C2 -> COMPRESSOR_PWM
- U1 pad 65: unconnected-(U1-PC8-Pad65) -> VALVE
- U1 pad 77: T2C1 -> STEPPER1_STEP
- U1 pad 79: PC11 -> USB_VSENSE
- U1 pad 82: U4T -> STEPPER_TX
- U1 pad 87: PD6 -> STEPPER1_DIR
- U1 pad 88: PD7 -> STEPPER2_DIR
- U1 pad 90: T3C1 alternativ zu C6 -> STEPPER2_STEP
- U1 pad 91: T3C2 -> STEPPER_EN
- U1 pad 97: U8R -> MALIBOTTI_RX
- U6 pad 4: I2C3_SDA -> I2C4_SDA
- U6 pad 5: I2C3_SCL -> I2C4_SCL
- U7 pad 14: STEPPER_UART -> STEPPER_RX
- U8 pad 14: STEPPER_UART -> STEPPER_RX
- U8 pad 16: STEPPER2_STEP_T3C2_T8C2 -> STEPPER2_STEP
- U8 pad 19: STEPPER2_DIR_T3C1_T8C1 -> STEPPER2_DIR
- U9 pad 1: +3.3VA -> /sensors/VA_HX711
Routing:
- net +3V3: track 40.8 -> 401.0 mm, vias 0 -> 30
- net 5-24V: track 0.00 -> 194.9 mm, vias 0 -> 11
- net +5V: track 0.00 -> 164.2 mm, vias 0 -> 3
- net GND: track 0.00 -> 118.4 mm, vias 0 -> 46
- net I2C1_SDA: track 0.00 -> 79.2 mm
- net +24V: track 0.00 -> 76.8 mm
- net ROBOT_RX: track 0.00 -> 75.5 mm, vias 0 -> 2
- net I2C1_SCL: track 0.00 -> 72.5 mm
- net unconnected-(U1-PC8-Pad65): track 59.6 -> 0.00 mm, vias 2 -> 0
- net STEPPER_EN: track 0.00 -> 55.4 mm, vias 0 -> 2
- net I2C4_SCL: track 0.00 -> 54.7 mm, vias 0 -> 2
- net STEPPER_RX: track 0.00 -> 54.2 mm, vias 0 -> 3
- net I2C4_SDA: track 18.4 -> 70.5 mm, vias 0 -> 4
- net MALIBOTTI_RX: track 0.00 -> 51.2 mm
- net VALVE: track 0.00 -> 50.7 mm
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- added copper zone on B.Cu, net GND
- added copper zone on F.Cu, net GND
- added copper zone on In1.Cu, net GND
- added copper zone on In2.Cu, net GND
Other:
- copper layers 2 -> 4

Commit message: WIP
Parts:
- added C62: u1, Capacitor_SMD:C_0402_1005Metric, F.Cu at (170.5, 77.4)
- added J24: WS2812_CH1, liebler_CONN:JST_XH_B3B-XH-A_1x03_P2.50mm_Vertical_smaller, B.Cu at (167.6, 67.2)
- added J25: WS2812_CH2, liebler_CONN:JST_XH_B3B-XH-A_1x03_P2.50mm_Vertical_smaller, B.Cu at (167.6, 61.0)
- added U11: 74AHCT125, Package_SO:SOIC-14_3.9x8.7mm_P1.27mm, F.Cu at (167.4, 73.2)
- moved R9 14.8 mm to (125.1, 99.5)
- moved R54 13.2 mm to (126.4, 99.7)
- moved R44 13.2 mm to (125.8, 100.8), turned to 90 degrees
- moved R8 13.0 mm to (125.1, 98.0)
- moved J11 10.7 mm to (183.5, 61.1)
- moved J10 10.7 mm to (183.5, 67.2)
- moved R10 7.00 mm to (117.9, 71.4)
- moved D1 7.00 mm to (114.1, 71.4)
- moved R4 4.67 mm to (105.1, 81.2), turned to 0 degrees
- moved C34 3.61 mm to (96.8, 68.9), turned to 90 degrees
- moved R5 2.86 mm to (106.4, 82.0), turned to 180 degrees
- moved TP1 2.79 mm to (119.8, 100.6)
- moved R7 2.44 mm to (108.8, 80.8), turned to -90 degrees
- moved R6 1.34 mm to (106.8, 81.0)
- moved R43 0.83 mm to (118.0, 99.4), turned to -45 degrees
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Connections:
- D1 pad 1: ADC1_IN11 -> LED_INFO
- U1 pad 46: PE15 -> LED_INFO
Routing:
- net +3V3: track 401.0 -> 317.4 mm
- net T15C1: track 0.00 -> 59.6 mm
- net T15C2: track 0.00 -> 55.9 mm
- net +5V: track 164.2 -> 195.7 mm, vias 3 -> 4
- net GND: track 118.4 -> 132.6 mm, vias 46 -> 40
- net I2C1_SCL: track 72.5 -> 84.4 mm
- net WS2812_CH2: track 0.00 -> 11.8 mm
- net I2C1_SDA: track 79.2 -> 90.0 mm
- net LED_INFO: track 0.00 -> 10.1 mm
- net STEPPER1_DIR: track 25.0 -> 20.7 mm
- net WS2812_CH1: track 0.00 -> 4.12 mm
- net STEPPER_RX: track 54.2 -> 51.2 mm
- net STEPPER_EN: track 55.4 -> 52.8 mm
- net Net-(C11-Pad1): track 28.9 -> 26.8 mm
- net ROBOT_RX: track 75.5 -> 77.0 mm
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- added copper zone on B.Cu, net +3V3
- added copper zone on F.Cu, net +3V3
