File: pcb_control_unit_ethernet/ethercat_esc.kicad_sch (KiCad schematic)
At the start: 37 parts, among them CN1 10p, U12 LAN9253_SIO_GPIO, X2 HR911105A_small, X3 HR911105A_small, Y2 25MHz

Commit message: WIP 2nd
Parts:
- removed RN1 (x2): 50R, Resistor_THT:R_Array_SIP5, symbol Device:R_Network04
- added R68, R69, R70, R71, R72, R73, R74, R75: 49R9, Resistor_SMD:R_0402_1005Metric, symbol Device:R
Connections:
- net RXNA: now also R68.2
- net RXNB: now also R72.2
- net RXPA: now also R69.2
- net RXPB: now also R73.2
- net TXNA: now also R70.2
- net TXNB: now also R74.2
- net TXPA: now also R71.2
- net TXPB: now also R75.2
- net at C80.1, L9.2, X2.4 (TCT)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: now also R68.1, R69.1, R70.1, R71.1, R72.1, R73.1, R74.1, R75.1
Other:
- moved on the sheet: L9

Commit message: Update ethercat_esc.kicad_sch
Parts:
- removed C72: u1, Capacitor_SMD:C_0201_0603Metric, symbol Device:C
- removed C73, C74, C75: 1u, Capacitor_SMD:C_0402_1005Metric, symbol Device:C
- removed L7, L8, L9: 600R@100M, Inductor_SMD:L_0603_1608Metric, symbol Device:L_Ferrite_Small
- removed R67: k33, Resistor_SMD:R_0402_1005Metric, symbol Device:R
- added C79, C81: u1, Capacitor_SMD:C_0201_0603Metric, symbol Device:C
- added C82, C83: 1u, Capacitor_SMD:C_0402_1005Metric, symbol Device:C
- added U13: ~, symbol liebler_SEMICONDUCTORS:LAN9253_SPI_GPIO_V2
- C71: value u1 -> 1u; footprint Capacitor_SMD:C_0201_0603Metric -> Capacitor_SMD:C_0402_1005Metric
- R?: renamed from R65; value 12k1 -> 4k7
- renumbered C63 to C?, C64 to C?, L6 to L?
Connections:
- net +3V3: now also L5.1, U13.14 (VDDIO), U13.20 (VDDIO), U13.32 (VDDIO), U13.37 (VDDIO), U13.47 (VDDIO), U13.5 (VDD33), U13.7 (REG_EN); no longer L?.2, U12.14 (VDDIO), U12.20 (VDDIO), U12.32 (VDDIO), U12.37 (VDDIO), U12.47 (VDDIO), U12.5 (VDD33), U12.7 (REG_EN)
- net ETHERCAT_IRQ: now also U13.44 (IRQ); no longer U12.44 (IRQ)
- net GND: now also C79.2, C81.2, C82.2, C83.2, U13.41 (TESTMODE_PULL_TO_GND); no longer U12.4 (OSCVSS), U12.41 (TESTMODE), U12.65 (VSS)
- net LINKACTLED0: now also U13.48 (LINKACTLED0/TDO/CHIP_MODE0/100FD_A/LEDPOL0); no longer U12.48 (LINKACTLED0/TDO/~{CHIP_MODE0}/~{100FD_A}/~{LEDPOL0})
- net LINKACTLED1: now also U13.46 (LINKACTLED1/TDI/CHIP_MODE1/LEDPOL1); no longer U12.46 (LINKACTLED1/TDI/~{CHIP_MODE1}/~{LEDPOL1})
- net QSPI_CLK: now also U13.19 (D9/AD9/LATCH_IN/SCK); no longer U12.19 (SCK)
- net QSPI_CS: now also U13.50 (D5/AD5/OUTVALID/SCS#); no longer U12.50 (SCS#)
- net QSPI_SIO0: now also U13.17 (D0/AD0/WD_STATE/SI/SIO0); no longer U12.17 (SI/SIO0)
- net QSPI_SIO1: now also U13.13 (D1/AD1/EOF/SO/SIO1); no longer U12.13 (SO/SIO1)
- net QSPI_SIO2: now also U13.12 (D2/AD2/SOF/SIO2/EE_EMUL_SPI0); no longer U12.12 (SIO2/~{EE_EMUL_SPI0})
- net QSPI_SIO3: now also U13.35 (D3/AD3/WD_TRIG/SIO3/EE_EMUL_SPI1); no longer U12.35 (SIO3/~{EE_EMUL_SPI1})
- net RUNLED: now also U13.45 (RUNLED/STATE_RUNLED/E2PSIZE/EE_EMUL0/LEDPOL3); no longer U12.45 (RUNLED/STATE_RUNLED/~{E2PSIZE}/~{EE_EMUL0}/~{LEDPOL3})
- net RXNA: now also U13.54 (RXNA); no longer U12.54 (RXNA)
- net RXNB: now also U13.61 (RXNB); no longer U12.61 (RXNB)
- net RXPA: now also U13.55 (RXPA); no longer U12.55 (RXPA)
- net RXPB: now also U13.60 (RXPB); no longer U12.60 (RXPB)
- net SYNC0: now also U13.34 (SYNC0/LATCH0/PME); no longer U12.34 (SYNC0/LATCH0/PME)
- net SYNC1: now also U13.18 (SYNC1/LATCH1/PME); no longer U12.18 (SYNC1/LATCH1/PME)
- net TXNA: now also U13.52 (TXNA); no longer U12.52 (TXNA)
- net TXNB: now also U13.61 (RXNB); no longer U12.63 (TXNB)
- net TXPA: now also U13.53 (TXPA); no longer U12.53 (TXPA)
- net TXPB: now also U13.62 (TXPB); no longer U12.62 (TXPB)
- net VDDCR_IN: no longer C68.1, C69.1, L5.2, U12.6 (VDDCR_OUT)
- net VDD33TXRX2: now reaches C80.1, R72.1, R73.1, R74.1, R75.1, X3.4 (TCT), X3.5 (RCT)
- net VDD33TXRX2: now also U13.64 (VDD33TXRX2); no longer R68.1, R69.1, R70.1, R71.1, X2.4 (TCT), X2.5 (RCT)
- net at C77.1, Y2.1: now also U13.1 (OSCI); no longer U12.1 (OSCI)
- net at C78.1, Y2.3: now also U13.2 (OSCO); no longer U12.2 (OSCO)
- net at R?.2: now also U13.8 (CLK_25/CLK_25_EN); no longer U12.57 (RBIAS)
- net ETHERCAT_RESET: now reaches C76.2, R64.2
- net ETHERCAT_RESET: now also U13.11 (~{RST}); no longer U12.11 (~{RST})
- net at U12.64 (VDD33TXRX2): no longer L?.1
- removed net +1V2: C71.1, L5.1, U12.56 (VDD12TX1), U12.59 (VDD12TX2)
- net SCL: no longer names the net of U12.43 (EESCL/TCK/~{EE_EMUL2})
- net SDA: no longer names the net of U12.42 (EESDA/TMS/~{EE_EMUL1})
- new net: C83.1, L5.2, U13.58 (VDD33BIAS)
- new net: R?.2, U13.66 (R_BIAS)
- new net EESCL: U13.43 (EESCL)
- new net EESDA: U13.42 (EESDA)
- new net ERRLED: U13.9 (ATEST/ERRLED/PME/100FD_B/LEDPOL4)
- new net VDD12TX1: C71.1, C79.1, C81.1, C82.1, L?.2, U13.56 (VDD12TX1), U13.59 (VDD12TX2)
- new net VDD33TXRX1: R68.1, R69.1, R70.1, R71.1, U13.51 (VDD33TXRX1), X2.4 (TCT), X2.5 (RCT)
- new net VDDCR: C68.1, C69.1, C?.1, C?.1, L?.1, U13.24 (VDDCR), U13.38 (VDDCR), U13.6 (VDDCR)
- new net VDDIO: U12.14 (VDDIO), U12.20 (VDDIO), U12.32 (VDDIO), U12.37 (VDDIO), U12.47 (VDDIO)
- no-connect marks 17 -> 0
Other:
- note added: "Check Document "EVB-LAN9253-ADD-ON Schematics""
- moved on the sheet: C68, C69, C76, C77, C78, L?, NT4, R64, R65, U12, Y2

Commit message: EtherCAT + HX711
Parts:
- added C? (x2): u1, Capacitor_SMD:C_0201_0603Metric, symbol Device:C
- added R?: 4k7, Resistor_SMD:R_0201_0603Metric, symbol Device:R
- R65: renamed from R?; value 4k7 -> 12k1
- gave numbers to parts that had none: 2
Connections:
- net GND: now also C?.2, C?.2, R?.1
- net VDDCR: now also C?.1, C?.1; no longer C63.1, C64.1
- net at U13.8 (CLK_25/CLK_25_EN): now also R?.2; no longer R65.2
