File: pcb_control_unit_ethercat/actors.kicad_sch (KiCad schematic)
At the start: 65 parts, among them J17 STEP1, J18 STEP2, J30 Valve, Q1 IRLML6344, Q2 IRLML6344, Q3 IRLML6344, Q5 IRLML6344, Q6 IRLML6344, U11 74AHCT125, U7 TMC2209, U8 TMC2209

Commit message: WIP
Parts:
- R40, R42: value 390m -> r1
- renumbered Conv1 to J19, Valve1 to J20, Robot1 to J21, Comp1 to J22, Valve2 to J31
Connections:
- net STEPPER_EN: no longer U7.2 (ENN), U8.2 (ENN)
- new net STEPPER1_EN: U7.2 (ENN), U8.2 (ENN)
Other:
- note added: "Es amago de querer controlar el paso de la senal"
- note added: "Stepper Driver 1 clasifier"
- note added: "Stepper Driver 2"
- note added: "Valve 2"
- note added: "Valve 3"
- note added: "la verdad no se de cuanto es el motor"
- note added: "steppers para ascensor y clasificador Motor DC es el conveyor"
- note removed: "Stepper Driver 1 elevator(600mA motor)"
- note removed: "Stepper Driver 2 clasifier (600mA motor)"
- note removed: "Valve 2 (for control loop)"
- note removed: "Valve 3 (for control loop)"
- note removed: "steppers for elevator and clasificator DC motor for conveyor"
- moved on the sheet: R40
Changed lines of the file:
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@@
 		)
 	)
-	(text "Valve 2 (for control loop)"
+	(text "Valve 2"
 		(exclude_from_sim no)
 		(at 157.48 54.61 0)
@@
 		)
 	)
+	(text "la verdad no se de cuanto\nes el motor"
+		(exclude_from_sim no)
+		(at 103.378 172.212 0)
+		(effects
+			(font
+				(size 1.27 1.27)
+				(color 255 0 0 1)
+			)
+		)
+	)
 	(text "Compressor"
 		(exclude_from_sim no)
@@
 		)
 	)
-	(text "Stepper Driver 2 clasifier (600mA motor)"
+	(text "Stepper Driver 2"
 		(exclude_from_sim no)
-		(at 42.926 98.806 0)
+		(at 30.48 99.314 0)
 		(effects
 			(font
@@
 		)
 	)
-	(text "steppers for elevator and clasificator\nDC motor for conveyor\n"
+	(text "steppers para ascensor y clasificador\nMotor DC es el conveyor\n"
 		(exclude_from_sim no)
 		(at 130.556 93.218 0)
@@
 		)
 	)
-	(text "Valve 3 (for control loop)"
+	(text "Valve 3"
 		(exclude_from_sim no)
 		(at 157.48 83.82 0)
@@
 		)
 	)
-	(text "Stepper Driver 1 elevator(600mA motor)\n"
+	(text "Stepper Driver 1 clasifier\n"
 		(exclude_from_sim no)
-		(at 42.926 14.732 0)
+		(at 34.29 15.24 0)
 		(effects
 			(font
@@
 		)
 	)
+	(text "Es amago de querer controlar \nel paso de la senal"
+		(exclude_from_sim no)
+		(at 154.94 123.444 0)
+		(effects
+			(font
+				(size 0.635 0.635)
+				(color 0 0 0 1)
+			)
+		)
+	)
 	(junction
 		(at 173.99 69.85)
@@
 	(wire
 		(pts
-			(xy 111.76 27.94) (xy 111.76 29.21)
+			(xy 111.76 26.67) (xy 111.76 29.21)
 		)
 		(stroke
@@
 	(wire
 		(pts
-			(xy 74.93 163.83) (xy 76.2 163.83)
+			(xy 74.93 163.83) (xy 77.47 163.83)
 		)
 		(stroke
@@
 	(wire
 		(pts
-			(xy 119.38 29.21) (xy 119.38 27.94)
+			(xy 119.38 29.21) (xy 119.38 26.67)
 		)
 		(stroke
@@
 		)
 	)
-	(global_label "STEPPER_EN"
+	(global_label "STEPPER1_EN"
 		(shape input)
 		(at 44.45 153.67 180)
@@
 		)
 		(property "Intersheetrefs" "${INTERSHEET_REFS}"
-			(at 29.7326 153.67 0)
+			(at 28.5231 153.67 0)
 			(effects
 				(font
@@
 	(global_label "STEPPER_RX"
 		(shape output)
-		(at 119.38 27.94 90)
+		(at 119.38 26.67 90)
 		(fields_autoplaced yes)
 		(effects
@@
 		)
 		(property "Intersheetrefs" "${INTERSHEET_REFS}"
-			(at 119.38 13.2226 90)
+			(at 119.38 11.9526 90)
 			(effects
 				(font
@@
 	(global_label "STEPPER_TX"
 		(shape input)
-		(at 111.76 27.94 90)
+		(at 111.76 26.67 90)
 		(fields_autoplaced yes)
 		(effects
@@
 		)
 		(property "Intersheetrefs" "${INTERSHEET_REFS}"
-			(at 111.76 13.525 90)
+			(at 111.76 12.255 90)
 			(effects
 				(font
@@
 		)
 	)
-	(global_label "STEPPER_EN"
+	(global_label "STEPPER1_EN"
 		(shape input)
 		(at 44.45 69.85 180)
@@
 		)
 		(property "Intersheetrefs" "${INTERSHEET_REFS}"
-			(at 29.7326 69.85 0)
+			(at 28.5231 69.85 0)
 			(effects
 				(font
@@
 		(dnp no)
 		(fields_autoplaced yes)
-		(property "Reference" "Robot1"
+		(property "Reference" "J21"
 			(at 229.87 97.7899 0)
 			(effects
@@
 			(project "pcb_control_unit_ethernet"
 				(path "/9c57264a-0988-4c94-95c0-340e4ca73bd5/3e57726e-e70f-48f8-bf8b-be1a55c6b2d5"
-					(reference "Robot1")
+					(reference "J21")
 					(unit 1)
 				)
@@
 	(symbol
 		(lib_id "Device:R")
-		(at 76.2 167.64 0)
+		(at 77.47 167.64 0)
 		(unit 1)
 		(exclude_from_sim no)
@@
 		(on_board yes)
 		(dnp no)
+		(fields_autoplaced yes)
 		(property "Reference" "R40"
-			(at 77.978 166.37 0)
+			(at 80.01 166.3699 0)
 			(effects
 				(font
@@
 			)
 		)
-		(property "Value" "390m"
-			(at 77.978 168.91 0)
+		(property "Value" "r1"
+			(at 80.01 168.9099 0)
 			(effects
 				(font
@@
 		)
 		(property "Footprint" "Resistor_SMD:R_1206_3216Metric"
-			(at 74.422 167.64 90)
+			(at 75.692 167.64 90)
 			(effects
 				(font
@@
 		)
 		(property "Datasheet" "~"
-			(at 76.2 167.64 0)
+			(at 77.47 167.64 0)
 			(effects
 				(font
@@
 		)
 		(property "Description" "Resistor"
-			(at 76.2 167.64 0)
+			(at 77.47 167.64 0)
 			(effects
 				(font
@@
 		)
 		(property "MPN" "FRM121WFR100TM"
-			(at 76.2 167.64 0)
+			(at 77.47 167.64 0)
 			(effects
 				(font
@@
 		)
 		(property "Manufacturer" " FOJAN"
-			(at 76.2 167.64 0)
+			(at 77.47 167.64 0)
 			(effects
 				(font
@@
 		(on_board yes)
 		(dnp no)
-		(property "Reference" "Comp1"
+		(property "Reference" "J22"
 			(at 233.426 53.594 0)
 			(effects
@@
 			(project "pcb_control_unit_ethernet"
 				(path "/9c57264a-0988-4c94-95c0-340e4ca73bd5/3e57726e-e70f-48f8-bf8b-be1a55c6b2d5"
-					(reference "Comp1")
+					(reference "J22")
 					(unit 1)
 				)
@@
 	(symbol
 		(lib_id "power:GND")
-		(at 76.2 171.45 0)
+		(at 77.47 171.45 0)
 		(unit 1)
 		(exclude_from_sim no)
@@
 		(fields_autoplaced yes)
 		(property "Reference" "#PWR0112"
-			(at 76.2 177.8 0)
+			(at 77.47 177.8 0)
 			(effects
 				(font
@@
 		)
 		(property "Value" "GND"
-			(at 76.2 176.53 0)
+			(at 77.47 176.53 0)
 			(effects
 				(font
@@
 		)
 		(property "Footprint" ""
-			(at 76.2 171.45 0)
+			(at 77.47 171.45 0)
 			(effects
 				(font
@@
 		)
 		(property "Datasheet" ""
-			(at 76.2 171.45 0)
+			(at 77.47 171.45 0)
 			(effects
 				(font
@@
 		)
 		(property "Description" "Power symbol creates a global label with name \"GND\" , ground"
-			(at 76.2 171.45 0)
+			(at 77.47 171.45 0)
 			(effects
 				(font
@@
 		(on_board yes)
 		(dnp no)
-		(property "Reference" "Conv1"
+		(property "Reference" "J19"
 			(at 146.05 57.404 0)
 			(effects
@@
 			(project "pcb_control_unit_ethernet"
 				(path "/9c57264a-0988-4c94-95c0-340e4ca73bd5/3e57726e-e70f-48f8-bf8b-be1a55c6b2d5"
-					(reference "Conv1")
+					(reference "J19")
 					(unit 1)
 				)
@@
 			)
 		)
-		(property "Value" "390m"
+		(property "Value" "r1"
 			(at 87.63 168.9099 0)
 			(effects
@@
 		(on_board yes)
 		(dnp no)
-		(property "Reference" "Valve1"
+		(property "Reference" "J20"
 			(at 185.166 29.21 0)
 			(effects
@@
 			(project "pcb_control_unit_ethernet"
 				(path "/9c57264a-0988-4c94-95c0-340e4ca73bd5/3e57726e-e70f-48f8-bf8b-be1a55c6b2d5"
-					(reference "Valve1")
+					(reference "J20")
 					(unit 1)
 				)
@@
 		(on_board yes)
 		(dnp no)
-		(property "Reference" "Valve2"
+		(property "Reference" "J31"
 			(at 185.166 57.15 0)
 			(effects
@@
 			(project "pcb_control_unit_ethernet"
 				(path "/9c57264a-0988-4c94-95c0-340e4ca73bd5/3e57726e-e70f-48f8-bf8b-be1a55c6b2d5"
-					(reference "Valve2")
+					(reference "J31")
 					(unit 1)
 				)
