File: pcb_control_unit_ethercat/pcb_control_unit_ethernet.kicad_sch (KiCad schematic)
At the start: 42 parts, among them J1 STDC14, J2 Micro_SD_Card_Det1, SW1 Reset, SW2 Boot, U1 STM32H563VITx, U10 SIT3051TK

Commit message: WIP
Parts:
- C1, C10, C14, C16, C2, C3, C4, C5, C6, C61, C7, C8: footprint Capacitor_SMD:C_0402_1005Metric -> Capacitor_SMD:C_0201_0603Metric
Connections:
- net COMPRESSOR_PWM: now also U1.61 (PD14); no longer U1.62 (PD15)
- net CONVEYOR_PWM: now also U1.62 (PD15); no longer U1.61 (PD14)
- net STEPPER_EN renamed STEPPER1_EN
Other:
- note added: "BD1 pero hay que conectarlo a CC1"
- note added: "DB2 pero hay que conectarlo a CC2"
- note added: "El sensor de peso se puede cambiar a NAU7802"
- note added: "Esto parece que esta bien NO TOCAR"
- note added: "Info para debugging y puede que para arranque"
- note added: "Para poder comunicarse por usb con un pc basicamente para debugear bien USart"
- note added: "QSPI es para etherCAT"
- note added: "Tranceptor CAN que se comunica con el stm y manda los datos a un conector que sirve para comunicarlo con componentes externos"
- note added: "Uart 7 Uart 12"
- note added: "comunicacion can"
- note added: "le quiere poner una pantallita"
- note added: "para conectar USB sense"
- note added: "se puede mover a cualquier GPIO"
- note added: "sensor Corriente"
- note added: "tiene que ser adc"
- note added: "tiene que ser este porque no usamos timer"
- note removed: "CAN BUS"
- note removed: "CAN Comunication"
- note removed: "CURRENT SENSOR"
- note removed: "DEBUGGER"
- note removed: "Extra SPI connection"
- note removed: "To connect to PC0"
- moved on the sheet: C61, D1, R10, R62, R63, U10
