File: pcb_control_unit_ethernet-2026-04-30_133407/pcb_control_unit_ethernet.kicad_pcb (KiCad board)
At the start: 4 copper layers, 188 x 65 mm, 267 parts, among them J1 STDC14, J2 Micro_SD_Card_Det1, J30 Valve, J5 USB STM32, J6 USB STM32, Q1 IRLML6344, Q2 IRLML6344, Q3 IRLML6344, Q4 MMBT4403, Q5 IRLML6344, Q6 IRLML6344, SW1 Reset, SW2 Boot, U1 STM32H563VITx, U10 SIT3051TK, U11 74AHCT125, U16 24LC512, U2 LAN8742A, U3 DCDC_MP2315, U4 TPS54202DDC, U5 AMS1117-3.3, U6 INA226, U7 TMC2209, U8 TMC2209, U9 HX711, X1 MT3608, Y1 25MHz, Y2 25MHz

Commit message: WIP
Parts:
- removed +24V: DC IN, Connector_BarrelJack:BarrelJack_Horizontal
- removed the C58 at (160.6, 75.6)
- removed the C58 at (214.3, 82.5)
- removed the C73 at (173.7, 59.5)
- removed C76: u1, Capacitor_SMD:C_0402_1005Metric
- removed C80: 10n, Capacitor_SMD:C_0603_1608Metric
- removed CanBus: CAN, liebler_CONN:JST_XH_B3B-XH-A_1x03_P2.50mm_Vertical_smaller
- removed Clasifier: STEP2, liebler_CONN:JST_XH_B4B-XH-A_1x04_P2.50mm_Vertical_smaller
- removed Comp: Compressor, liebler_CONN:PhoenixContact_MC_1,5_2-G-3.5_1x02_P3.50mm_Horizontal_smallerCourtyard
- removed Conv: Conveyor, liebler_CONN:PhoenixContact_MC_1,5_2-G-3.5_1x02_P3.50mm_Horizontal_smallerCourtyard
- removed Elevator: STEP1, liebler_CONN:JST_XH_B4B-XH-A_1x04_P2.50mm_Vertical_smaller
- removed EthercatA, EthercatB: HR911105A_small, liebler_CONN:RJ45_HANRUN_HR911105A
- removed I2C1A: RGB, liebler_CONN:JST_XH_B5B-XH-A_1x05_P2.50mm_Vertical_smaller
- removed I2C1B: TOF1, liebler_CONN:JST_XH_B5B-XH-A_1x05_P2.50mm_Vertical_smaller
- removed Malibotti: Malibotti, liebler_CONN:JST_XH_B4B-XH-A_1x04_P2.50mm_Vertical_smaller
- removed Pressure: PressureTransducer, liebler_CONN:JST_XH_B3B-XH-A_1x03_P2.50mm_Vertical_smaller
- removed R87, R88: 10k, Resistor_SMD:R_0201_0603Metric
- removed Robot: Bus-Servo, Connector_Molex:Molex_SPOX_5267-03A_1x03_P2.50mm_Vertical
- removed Valve: Valve, liebler_CONN:PhoenixContact_MC_1,5_2-G-3.5_1x02_P3.50mm_Horizontal_smallerCourtyard
- removed Weightcell A: Weight, liebler_CONN:JST_XH_B4B-XH-A_1x04_P2.50mm_Vertical_smaller
- removed Weightcell B: INB, Connector_JST:JST_XH_B2B-XH-A_1x02_P2.50mm_Vertical
- added C58: u1, Capacitor_SMD:C_0402_1005Metric, F.Cu at (200.3, 73.0)
- added C70: u1, Capacitor_SMD:C_0402_1005Metric, F.Cu at (202.4, 87.2)
- added CanBus1: CAN, liebler_CONN:JST_XH_B3B-XH-A_1x03_P2.50mm_Vertical_smaller, B.Cu at (112.2, 105.5)
- added Comp1: Compressor, liebler_CONN:PhoenixContact_MC_1,5_2-G-3.5_1x02_P3.50mm_Horizontal_smallerCourtyard, B.Cu at (78.9, 65.6)
- added Conv1: Conveyor, liebler_CONN:PhoenixContact_MC_1,5_2-G-3.5_1x02_P3.50mm_Horizontal_smallerCourtyard, B.Cu at (87.5, 65.6)
- added EthercatA1: HR911105A_small, liebler_CONN:RJ45_HANRUN_HR911105A, B.Cu at (218.3, 68.4)
- added EthercatB1: HR911105A_small, liebler_CONN:RJ45_HANRUN_HR911105A, B.Cu at (199.7, 68.4)
- added I2C1A1: RGB, liebler_CONN:JST_XH_B5B-XH-A_1x05_P2.50mm_Vertical_smaller, B.Cu at (182.7, 61.1)
- added I2C1B1: TOF1, liebler_CONN:JST_XH_B5B-XH-A_1x05_P2.50mm_Vertical_smaller, B.Cu at (182.7, 67.2)
- added J17: STEP1, liebler_CONN:JST_XH_B4B-XH-A_1x04_P2.50mm_Vertical_smaller, B.Cu at (142.5, 117.0)
- added J18: STEP2, liebler_CONN:JST_XH_B4B-XH-A_1x04_P2.50mm_Vertical_smaller, B.Cu at (155.3, 117.0)
- added J23: Weight, liebler_CONN:JST_XH_B4B-XH-A_1x04_P2.50mm_Vertical_smaller, B.Cu at (156.2, 67.2)
- added J3: INB, Connector_JST:JST_XH_B2B-XH-A_1x02_P2.50mm_Vertical, B.Cu at (152.8, 73.8)
- added J4: DC IN, Connector_BarrelJack:BarrelJack_Horizontal, B.Cu at (101.2, 108.5)
- added Malibotti1: Malibotti, liebler_CONN:JST_XH_B4B-XH-A_1x04_P2.50mm_Vertical_smaller, B.Cu at (156.2, 61.1)
- added Pressure1: PressureTransducer, liebler_CONN:JST_XH_B3B-XH-A_1x03_P2.50mm_Vertical_smaller, B.Cu at (127.4, 60.0)
- added Robot1: Bus-Servo, Connector_Molex:Molex_SPOX_5267-03A_1x03_P2.50mm_Vertical, B.Cu at (173.2, 120.1)
- added Valve1: Valve, liebler_CONN:PhoenixContact_MC_1,5_2-G-3.5_1x02_P3.50mm_Horizontal_smallerCourtyard, B.Cu at (70.4, 65.6)
- R1, R11, R12, R13, R14, R15, R16, R17, R18, R19, R2, R20, R21, R22, R23, R24, R3, R35, R36, R4, R44, R46, R5, R6, R63, R64, R65, R67, R7, R8, R89, R9: footprint Resistor_SMD:R_0201_0603Metric -> Resistor_SMD:R_0402_1005Metric
- R34: footprint Resistor_SMD:R_2010_5025Metric -> Resistor_SMD:R_1206_3216Metric
- moved R8 62.5 mm to (180.6, 69.3), turned to 90 degrees
- moved R9 61.9 mm to (179.1, 69.0), turned to 180 degrees
- moved D6 32.1 mm to (223.5, 82.0), turned to 0 degrees
- moved R77 29.6 mm to (219.8, 82.0), turned to 180 degrees
- moved R78 29.5 mm to (218.2, 81.5), turned to -90 degrees
- moved R44 27.5 mm to (153.1, 104.5)
- moved R54 24.7 mm to (116.1, 77.2)
- moved L9 23.8 mm to (199.0, 72.4), turned to -90 degrees
- moved C73 18.9 mm to (216.8, 79.0), turned to -90 degrees
- moved C85 18.2 mm to (216.3, 97.0), turned to -90 degrees
- moved R46 15.2 mm to (140.6, 106.1), turned to 0 degrees
- moved R6 15.1 mm to (107.7, 65.9), turned to -90 degrees
- moved C68 12.3 mm to (202.4, 88.1), turned to 180 degrees
- moved L3 10.4 mm to (80.1, 94.8)
- moved R80 10.3 mm to (192.7, 84.5), turned to 0 degrees
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- renumbered C70 to C73, ETHERNET to ETHERNET1
Connections:
- C73 pad 1: +3V3 -> /EtherCAT/VDD33TXRX1
- C74 pad 1: /EtherCAT/VDD33TXRX1 -> /EtherCAT/VDD33TXRX2
- L9 pad 2: /EtherCAT/VDD33TXRX1 -> /EtherCAT/VDD33TXRX2
- U1 pad 61: COMPRESSOR_PWM -> CONVEYOR_PWM
- U1 pad 62: CONVEYOR_PWM -> COMPRESSOR_PWM
- U1 pad 8: PC14 -> ETHERCAT_RESET
- U1 pad 93: STEPPER1_EN -> STEPPER_EN
- U7 pad 2: STEPPER1_EN -> STEPPER_EN
- U8 pad 2: STEPPER1_EN -> STEPPER_EN
- Y2 pad 1: Net-(U13A-OSCI) -> Net-(U13A-OSCO)
- Y2 pad 3: Net-(U13A-OSCO) -> Net-(U13A-OSCI)
Routing:
- net ETHERCAT_RESET: track 2.04 -> 82.6 mm, vias 0 -> 2
- net STEPPER_EN: track 0.00 -> 67.2 mm, vias 0 -> 2
- net STEPPER1_EN: track 67.2 -> 0.00 mm, vias 4 -> 0
- net RUNLED: track 40.0 -> 10.8 mm, vias 2 -> 0
- net USBPD_CC2: track 77.3 -> 57.1 mm
- net GND: track 142.8 -> 122.8 mm, vias 359 -> 453
- net T15C2: track 58.0 -> 72.2 mm
- net SD_CMD: track 36.1 -> 22.3 mm, vias 0 -> 2
- net SPI4_MOSI: track 114.1 -> 100.4 mm, vias 1 -> 2
- net QSPI_CLK: track 113.1 -> 99.4 mm
- net QSPI_CS: track 155.7 -> 143.3 mm, vias 6 -> 4
- net VALVE3: track 69.9 -> 58.1 mm
- net QSPI_SIO1: track 106.4 -> 94.7 mm
- net SD_D0: track 50.9 -> 39.4 mm
- net 5-24V: track 178.1 -> 167.2 mm, vias 14 -> 33
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- added copper zone on B.Cu, net 5-24V
- added copper zone on F.Cu, net 5-24V

Commit message: WIP
Parts:
- removed C25, C26: 10n, Capacitor_SMD:C_0603_1608Metric
- removed R19, R21, R22, R23: 10k, Resistor_SMD:R_0402_1005Metric
- added C75: 22n/50V, Capacitor_SMD:C_0402_1005Metric, F.Cu at (141.4, 73.2)
- added R76: 33R, Resistor_SMD:R_0402_1005Metric, F.Cu at (129.3, 81.3)
- C17, C19: value 5p6 -> 22p
- C18: value u1 -> 10n; footprint Capacitor_SMD:C_0201_0603Metric -> Capacitor_SMD:C_0402_1005Metric
- C22, C23: value u1 -> 10n
- R20: value 10k -> 2k2
- R29, R30: value k33 -> 330
- R83, R84: value 2.2k -> 2k2
- moved R15 29.9 mm to (149.7, 63.6), turned to 0 degrees
- moved R8 12.0 mm to (176.5, 80.6), turned to 0 degrees
- moved R10 10.8 mm to (108.3, 76.4), turned to -90 degrees
- moved R9 8.20 mm to (178.4, 77.2)
- moved D1 5.36 mm to (110.0, 74.5), turned to 180 degrees
- moved R29 3.80 mm to (138.8, 63.6), turned to 0 degrees
- moved SW2 1.55 mm to (128.1, 98.4)
- moved L2 1.49 mm to (134.6, 79.2)
- moved C24 1.47 mm to (136.1, 79.2)
- moved R18 1.43 mm to (126.5, 77.1)
- moved R3 1.23 mm to (133.2, 100.5)
- moved R16 1.03 mm to (126.5, 75.2)
- moved C33 0.75 mm to (100.2, 83.3)
- moved C67 0.64 mm to (203.3, 92.5)
- moved R64 0.55 mm to (199.5, 90.0)
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Connections:
- ETHERNET1 pad 12: +3V3 -> /eth/LED2
- ETHERNET1 pad 4: Net-(ETHERNET1-RCT) -> /eth/ETH_VA
- ETHERNET1 pad 5: Net-(ETHERNET1-RCT) -> /eth/ETH_VA
- ETHERNET1 pad 9: +3V3 -> /eth/LED1
- R15 pad 1: Net-(U2-RXER/PHYAD0) -> /eth/LED2
- R29 pad 2: /eth/LED1 -> GND
- R30 pad 2: /eth/LED2 -> GND
- U2 pad 10: Net-(U2-RXER/PHYAD0) -> unconnected-(U2-RXER/PHYAD0-Pad10)
- U2 pad 14: ETH_REF_CLK -> Net-(U2-~{INT}/REFCLKO)
Routing:
- net GND: track 122.8 -> 213.2 mm, vias 453 -> 516
- net +3V3: track 534.7 -> 503.8 mm, vias 70 -> 65
- net /eth/ETH_VA: track 20.6 -> 31.2 mm
- net Net-(ETHERNET1-RCT): track 6.75 -> 0.00 mm
- net /eth/LED2: track 19.0 -> 25.4 mm
- net +5V: track 190.4 -> 196.5 mm, vias 8 -> 9
- net ETH_MDC: track 20.7 -> 14.6 mm
- net Net-(U2-RXER/PHYAD0): track 5.01 -> 0.00 mm
- net Net-(C77-Pad2): track 15.5 -> 20.3 mm
- net LED_INFO: track 11.1 -> 6.51 mm
- net SD_CMD: track 22.3 -> 17.9 mm
- net PRESSURE_ADC: track 24.6 -> 20.4 mm
- net /EtherCAT/VDD12TX1: track 11.1 -> 14.5 mm
- net ETH_REF_CLK: track 9.95 -> 6.66 mm
- net /EtherCAT/VDD33TXRX2: track 22.3 -> 25.6 mm
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Other:
- board text added: "+-Sig"
- board text added: "+VALVE1-"
- board text added: "+VALVE2-"
- board text added: "----"
- board text added: "ADC"
- board text added: "INFO LED"
- board text added: "Pressure Sns"
- board text added: "Sorter"
- board text added: "Stepper 1"
- board text added: "Stepper 2"
- board text added: "WeightCell"
- board text removed: "+ VALVE -"
- board text removed: "-------"
- board text removed: "CTRL 1"
- board text removed: "CTRL 2"
- board text removed: "Clasifier"
- board text removed: "SCL SDA IRQ3 GND 3V3"
- board text removed: "k1"
- board text removed: "sensor"
