File: pcb_control_unit_ethernet-2026-04-30_133407/conn.kicad_sch (KiCad schematic)
At the start: 21 parts, among them J6 USB STM32

Commit message: WIP
Parts:
- R35, R36: footprint Resistor_SMD:R_0201_0603Metric -> Resistor_SMD:R_0402_1005Metric
Changed lines of the file:
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@@
 			)
 		)
-		(property "Footprint" "Resistor_SMD:R_0201_0603Metric"
+		(property "Footprint" "Resistor_SMD:R_0402_1005Metric"
 			(at 44.45 28.448 90)
 			(effects
@@
 			)
 		)
-		(property "Footprint" "Resistor_SMD:R_0201_0603Metric"
+		(property "Footprint" "Resistor_SMD:R_0402_1005Metric"
 			(at 44.45 30.988 90)
 			(effects
