File: pcb_control_unit_ethernet-2026-04-30_133407/eth.kicad_sch (KiCad schematic)
At the start: 31 parts, among them U2 LAN8742A, Y1 25MHz

Commit message: WIP
Parts:
- R15, R16, R17, R18, R19, R20, R21, R22, R23, R24: footprint Resistor_SMD:R_0201_0603Metric -> Resistor_SMD:R_0402_1005Metric
Changed lines of the file:
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@@
 			)
 		)
-		(property "Footprint" "Resistor_SMD:R_0201_0603Metric"
+		(property "Footprint" "Resistor_SMD:R_0402_1005Metric"
 			(at 65.532 97.79 90)
 			(effects
@@
 			)
 		)
-		(property "Footprint" "Resistor_SMD:R_0201_0603Metric"
+		(property "Footprint" "Resistor_SMD:R_0402_1005Metric"
 			(at 127 81.788 90)
 			(effects
@@
 			)
 		)
-		(property "Footprint" "Resistor_SMD:R_0201_0603Metric"
+		(property "Footprint" "Resistor_SMD:R_0402_1005Metric"
 			(at 57.15 74.168 90)
 			(effects
@@
 			)
 		)
-		(property "Footprint" "Resistor_SMD:R_0201_0603Metric"
+		(property "Footprint" "Resistor_SMD:R_0402_1005Metric"
 			(at 59.69 79.248 90)
 			(effects
@@
 			)
 		)
-		(property "Footprint" "Resistor_SMD:R_0201_0603Metric"
+		(property "Footprint" "Resistor_SMD:R_0402_1005Metric"
 			(at 61.722 97.79 90)
 			(effects
@@
 			)
 		)
-		(property "Footprint" "Resistor_SMD:R_0201_0603Metric"
+		(property "Footprint" "Resistor_SMD:R_0402_1005Metric"
 			(at 64.262 60.96 90)
 			(effects
@@
 			)
 		)
-		(property "Footprint" "Resistor_SMD:R_0201_0603Metric"
+		(property "Footprint" "Resistor_SMD:R_0402_1005Metric"
 			(at 57.15 71.628 90)
 			(effects
@@
 			)
 		)
-		(property "Footprint" "Resistor_SMD:R_0201_0603Metric"
+		(property "Footprint" "Resistor_SMD:R_0402_1005Metric"
 			(at 33.782 78.74 90)
 			(effects
@@
 			)
 		)
-		(property "Footprint" "Resistor_SMD:R_0201_0603Metric"
+		(property "Footprint" "Resistor_SMD:R_0402_1005Metric"
 			(at 60.452 60.96 90)
 			(effects
@@
 			)
 		)
-		(property "Footprint" "Resistor_SMD:R_0201_0603Metric"
+		(property "Footprint" "Resistor_SMD:R_0402_1005Metric"
 			(at 68.072 60.96 90)
 			(effects

Commit message: WIP
Parts:
- removed C25, C26: 10n, Capacitor_SMD:C_0603_1608Metric, symbol Device:C
- removed R19, R21, R22, R23: 10k, Resistor_SMD:R_0402_1005Metric, symbol Device:R
- added C75: 22n/50V, Capacitor_SMD:C_0402_1005Metric, symbol Device:C
- added R76: 33R, Resistor_SMD:R_0402_1005Metric, symbol Device:R
- C17, C19: value 5p6 -> 22p
- C18: value u1 -> 10n; footprint Capacitor_SMD:C_0201_0603Metric -> Capacitor_SMD:C_0402_1005Metric
- C22, C23: value u1 -> 10n
- R20: value 10k -> 2k2
- R29, R30: value k33 -> 330
Connections:
- net +3V3: no longer ETHERNET1.12, ETHERNET1.9
- net ETH_REF_CLK: now also R76.1; no longer U2.14 (~{INT}/REFCLKO)
- net ETH_VA: now also ETHERNET1.4 (TCT), ETHERNET1.5 (RCT), C75.1
- net GND: now also R29.2, R30.2, C75.2
- net LED1: now also ETHERNET1.9; no longer R29.2
- net LED2: now also ETHERNET1.12, R15.1; no longer R30.2
- net at U2.10 (RXER/PHYAD0): no longer R15.1
- new net: R76.2, U2.14 (~{INT}/REFCLKO)
- no-connect marks 0 -> 1
Other:
- note added: "Capacitor close to RCT"
- note added: "REFCLO Functionality selected for Pin 14"
- note added: "WPD"
- note added: "WPU"
- note added: "u1 on each side of Ferrite Bead"

Commit message: WIP
Parts:
- C24: footprint Capacitor_SMD:C_0603_1608Metric -> Capacitor_SMD:C_0805_2012Metric
- L2: value 600R@100M -> 220R@100M
- R20: value 2k2 -> 3k3
