File: pcb_control_unit_ethernet-2026-04-30_133407/psu.kicad_sch (KiCad schematic)
At the start: 24 parts, among them J4 DC IN, J5 USB STM32, U3 DCDC_MP2315, U4 TPS54202DDC, U5 AMS1117-3.3, U6 INA226, X1 MT3608

Commit message: WIP
Parts:
- removed R87, R88: 10k, Resistor_SMD:R_0201_0603Metric, symbol Device:R
- R34: footprint Resistor_SMD:R_2010_5025Metric -> Resistor_SMD:R_1206_3216Metric
- R89: footprint Resistor_SMD:R_0201_0603Metric -> Resistor_SMD:R_0402_1005Metric
Changed lines of the file:
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@@
 	)
 	(junction
-		(at 207.01 27.94)
-		(diameter 0)
-		(color 0 0 0 0)
-	)
-	(junction
 		(at 194.31 27.94)
 		(diameter 0)
@@
 	)
 	(junction
-		(at 212.09 27.94)
-		(diameter 0)
-		(color 0 0 0 0)
-	)
-	(junction
 		(at 124.46 82.55)
 		(diameter 0)
@@
 	(wire
 		(pts
-			(xy 207.01 27.94) (xy 212.09 27.94)
-		)
-		(stroke
-			(width 0)
-			(type default)
-		)
-	)
-	(wire
-		(pts
 			(xy 212.09 35.56) (xy 212.09 48.26)
 		)
@@
 	(wire
 		(pts
-			(xy 194.31 27.94) (xy 207.01 27.94)
-		)
-		(stroke
-			(width 0)
-			(type default)
-		)
-	)
-	(wire
-		(pts
 			(xy 66.04 19.05) (xy 66.04 24.13)
 		)
@@
 	(wire
 		(pts
-			(xy 212.09 27.94) (xy 217.17 27.94)
+			(xy 194.31 27.94) (xy 217.17 27.94)
 		)
 		(stroke
@@
 			)
 		)
-		(property "Footprint" "Resistor_SMD:R_0201_0603Metric"
+		(property "Footprint" "Resistor_SMD:R_0402_1005Metric"
 			(at 215.392 31.75 90)
 			(effects
@@
 	)
 	(symbol
-		(lib_id "Device:R")
-		(at 207.01 31.75 0)
-		(unit 1)
-		(exclude_from_sim no)
-		(in_bom yes)
-		(on_board yes)
-		(dnp no)
-		(property "Reference" "R87"
-			(at 204.724 33.274 90)
-			(effects
-				(font
-					(size 1.27 1.27)
-				)
-				(justify left)
-			)
-		)
-		(property "Value" "10k"
-			(at 207.01 33.528 90)
-			(effects
-				(font
-					(size 1.27 1.27)
-				)
-				(justify left)
-			)
-		)
-		(property "Footprint" "Resistor_SMD:R_0201_0603Metric"
-			(at 205.232 31.75 90)
-			(effects
-				(font
-					(size 1.27 1.27)
-				)
-				(hide yes)
-			)
-		)
-		(property "Datasheet" "~"
-			(at 207.01 31.75 0)
-			(effects
-				(font
-					(size 1.27 1.27)
-				)
-				(hide yes)
-			)
-		)
-		(property "Description" "Resistor"
-			(at 207.01 31.75 0)
-			(effects
-				(font
-					(size 1.27 1.27)
-				)
-				(hide yes)
-			)
-		)
-		(pin "2"
-		)
-		(pin "1"
-		)
-		(instances
-			(project "pcb_control_unit_ethernet"
-				(path "/9c57264a-0988-4c94-95c0-340e4ca73bd5/ed06edb5-031f-42a3-ad58-55ca73c66f14"
-					(reference "R87")
-					(unit 1)
-				)
-			)
-		)
-	)
-	(symbol
 		(lib_id "Device:C")
 		(at 55.88 22.86 180)
@@
 	)
 	(symbol
-		(lib_id "Device:R")
-		(at 212.09 31.75 0)
-		(unit 1)
-		(exclude_from_sim no)
-		(in_bom yes)
-		(on_board yes)
-		(dnp no)
-		(property "Reference" "R88"
-			(at 210.058 33.528 90)
-			(effects
-				(font
-					(size 1.27 1.27)
-				)
-				(justify left)
-			)
-		)
-		(property "Value" "10k"
-			(at 212.09 33.528 90)
-			(effects
-				(font
-					(size 1.27 1.27)
-				)
-				(justify left)
-			)
-		)
-		(property "Footprint" "Resistor_SMD:R_0201_0603Metric"
-			(at 210.312 31.75 90)
-			(effects
-				(font
-					(size 1.27 1.27)
-				)
-				(hide yes)
-			)
-		)
-		(property "Datasheet" "~"
-			(at 212.09 31.75 0)
-			(effects
-				(font
-					(size 1.27 1.27)
-				)
-				(hide yes)
-			)
-		)
-		(property "Description" "Resistor"
-			(at 212.09 31.75 0)
-			(effects
-				(font
-					(size 1.27 1.27)
-				)
-				(hide yes)
-			)
-		)
-		(pin "2"
-		)
-		(pin "1"
-		)
-		(instances
-			(project "pcb_control_unit_ethernet"
-				(path "/9c57264a-0988-4c94-95c0-340e4ca73bd5/ed06edb5-031f-42a3-ad58-55ca73c66f14"
-					(reference "R88")
-					(unit 1)
-				)
-			)
-		)
-	)
-	(symbol
 		(lib_id "Device:C")
 		(at 90.17 27.94 0)
@@
 			)
 		)
-		(property "Footprint" "Resistor_SMD:R_2010_5025Metric"
+		(property "Footprint" "Resistor_SMD:R_1206_3216Metric"
 			(at 174.752 49.53 90)
 			(effects

Commit message: WIP
Parts:
- removed U3: DCDC_MP2315, liebler_MODULES:DCDC_MP2315, symbol liebler_MODULES:DCDC_MP2315
- added C76: u1/35V, Capacitor_SMD:C_0805_2012Metric, symbol Device:C
- added C80: 10u/35V, Capacitor_SMD:C_0805_2012Metric, symbol Device:C
- added C84: u1/16V, Capacitor_SMD:C_0402_1005Metric, symbol Device:C
- added C88: 56p, Capacitor_SMD:C_0402_1005Metric, symbol Device:C
- added C89, C98: 22u, Capacitor_SMD:C_0805_2012Metric, symbol Device:C
- added L10: 12uH, Inductor_SMD:L_Abracon_ASPI-0630LR, symbol Device:L
- added R87: 5k1, Resistor_SMD:R_0402_1005Metric, symbol Device:R
- added R88: M1, Resistor_SMD:R_0402_1005Metric, symbol Device:R
- added R96: 330, Resistor_SMD:R_0402_1005Metric, symbol Device:R
- added U12: TPS54202DDC, Package_TO_SOT_SMD:SOT-23-6_Handsoldering, symbol Regulator_Switching:TPS54202DDC
- C27: footprint Capacitor_SMD:C_0603_1608Metric -> Capacitor_SMD:C_0805_2012Metric
- C29: footprint Capacitor_SMD:C_0603_1608Metric -> Capacitor_SMD:C_0402_1005Metric
- L3: value 10uH -> 12uH
- U6: footprint Package_SO:VSSOP-10_3x3mm_P0.5mm -> Package_SO:TSSOP-10_3x3mm_P0.5mm
Connections:
- net 5-24V: now also C76.2, C80.2, U12.3 (VIN)
- net GND: now also C76.1, C80.1, C89.2, C98.2, R87.1, U12.1 (GND)
- new net: R87.2, R96.1
- new net +12V: C88.2, C89.1, C98.1, L10.1, R88.1
- new net BOOT12: C84.1, U12.6 (BOOT)
- new net FB12: C88.1, R88.2, R96.2, U12.4 (FB)
- new net SW12: C84.2, L10.2, U12.2 (SW)
Other:
- note added: "PSU 12V"
- note added: "PSU 5V"
- note removed: "9V - 5-24V"
- note removed: "PSU"
