File: pcb_control_unit_ethernet-2026-04-30_133407/sensors.kicad_sch (KiCad schematic)
At the start: 17 parts, among them J23 Weight, J3 INB, Q4 MMBT4403, U9 HX711

Commit message: WIP
Parts:
- C55, C60: footprint Capacitor_SMD:C_0805_2012Metric_Pad1.18x1.45mm_HandSolder -> Capacitor_SMD:C_0805_2012Metric
- L4: footprint Inductor_SMD:L_0805_2012Metric_Pad1.05x1.20mm_HandSolder -> Inductor_SMD:L_0805_2012Metric
- L6: value 600R@100M -> 220R@100M
