File: pcb_control_unit_ethernet-2026-04-30_133407/actors.kicad_sch (KiCad schematic)
At the start: 65 parts, among them J17 STEP1, J18 STEP2, J30 Valve, Q1 IRLML6344, Q2 IRLML6344, Q3 IRLML6344, Q5 IRLML6344, Q6 IRLML6344, U11 74AHCT125, U7 TMC2209, U8 TMC2209

Commit message: WIP
Parts:
- R44, R46: footprint Resistor_SMD:R_0201_0603Metric -> Resistor_SMD:R_0402_1005Metric
Connections:
- net STEPPER1_EN is gone; now on net STEPPER_EN: U7.2 (ENN), U8.2 (ENN)
Changed lines of the file:
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@@
 		)
 	)
-	(global_label "STEPPER1_EN"
+	(global_label "STEPPER_EN"
 		(shape input)
 		(at 44.45 153.67 180)
@@
 		)
 		(property "Intersheetrefs" "${INTERSHEET_REFS}"
-			(at 28.5231 153.67 0)
+			(at 29.7326 153.67 0)
 			(effects
 				(font
@@
 		)
 	)
-	(global_label "STEPPER1_EN"
+	(global_label "STEPPER_EN"
 		(shape input)
 		(at 44.45 69.85 180)
@@
 		)
 		(property "Intersheetrefs" "${INTERSHEET_REFS}"
-			(at 28.5231 69.85 0)
+			(at 29.7326 69.85 0)
 			(effects
 				(font
@@
 			)
 		)
-		(property "Footprint" "Resistor_SMD:R_0201_0603Metric"
+		(property "Footprint" "Resistor_SMD:R_0402_1005Metric"
 			(at 126.492 27.94 90)
 			(effects
@@
 			)
 		)
-		(property "Footprint" "Resistor_SMD:R_0201_0603Metric"
+		(property "Footprint" "Resistor_SMD:R_0402_1005Metric"
 			(at 122.682 27.94 90)
 			(effects

Commit message: WIP
Parts:
- C36, C37: value u1 -> u1/50V
Connections:
- net +9V renamed +12V
- net VALVE renamed VALVE1

Commit message: Release Candidate
Connections:
- net T15C1 renamed WS2812_1
- net T15C2 renamed WS2812_2
Changed lines of the file:
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@@
 		)
 	)
-	(global_label "T15C1"
+	(global_label "WS2812_1"
 		(shape input)
 		(at 129.54 114.3 180)
@@
 		)
 		(property "Intersheetrefs" "${INTERSHEET_REFS}"
-			(at 120.6887 114.3 0)
+			(at 116.8788 114.3 0)
 			(hide yes)
 			(show_name no)
@@
 		)
 	)
-	(global_label "T15C2"
+	(global_label "WS2812_2"
 		(shape input)
 		(at 129.54 133.35 180)
@@
 		)
 		(property "Intersheetrefs" "${INTERSHEET_REFS}"
-			(at 120.6887 133.35 0)
-			(hide yes)
-			(show_name no)
+			(at 116.8788 133.35 0)
+			(hide yes)
+			(show_name no)
