File: pcb_factory_control_unit/pcb_factory_control_unit.kicad_pcb (KiCad board)
At the start: 4 copper layers, 188 x 65 mm, 274 parts, among them J1 STDC14, J17 STEP1, J18 STEP2, J2 Micro_SD_Card_Det1, J23 Weight, J3 INB, J30 Valve, J4 DC IN, J5 USB STM32, J6 USB STM32, Q1 IRLML6344, Q2 IRLML6344, Q3 IRLML6344, Q4 MMBT4403, Q5 IRLML6344, Q6 IRLML6344, SW1 Reset, SW2 Boot, U1 STM32H563VITx, U10 SIT3051TK, U11 74AHCT125, U12 TPS54202DDC, U16 24LC512, U2 LAN8742A, U4 TPS54202DDC, U5 AMS1117-3.3, U6 INA226, U7 TMC2209, U8 TMC2209, U9 HX711, X1 MT3608, Y1 25MHz, Y2 25MHz

Commit message: Changed LED ReverseMount Footprint, Removed PullUp, HSOS Logo
Parts:
- added G***: LOGO, liebler_DRAWINGS:LOGO_FHOS_50mm, B.Cu at (156.0, 93.1)
- D1, D2, D3, D4, D5, D6, D7, D8: footprint liebler_OPTO:LED_1206_3216Metric_ReverseMount -> LED_SMD:LED_1206_3216Metric_ReverseMount_Hole1.8x2.4mm
- moved R80 1.35 mm to (186.0, 84.0)
- moved R78 0.94 mm to (218.7, 84.0)
- moved R79 0.73 mm to (188.0, 84.0), turned to 180 degrees
- moved R10 0.57 mm to (107.9, 76.8)
- moved X1 0.40 mm to (85.0, 89.6)
- moved R77 0.38 mm to (216.8, 84.0), turned to 0 degrees
- moved D1 0.12 mm to (110.0, 74.4)
Routing:
- net GND: track 834.8 -> 843.2 mm, vias 477 -> 474
- net ERRLED: track 14.1 -> 16.0 mm
- net +3V3: track 526.1 -> 524.4 mm
- net +24V: track 155.7 -> 154.5 mm
- net 5-24V: track 201.3 -> 200.3 mm
- net RUNLED: track 10.9 -> 11.6 mm
- net Net-(D6-K): track 1.47 -> 2.12 mm
- net Net-(D7-K): track 1.41 -> 2.02 mm
- net Net-(D1-A): track 1.34 -> 1.92 mm
Other:
- board text added: "Factory-in-a-Box Control Unit v1.1"
- board text added: "github.com/klaus-liebler/factory_in_a_box (c) Klaus Liebler 2026-07-14"
- board text removed: "(c) Danielo Miguel (c) Klaus Liebler 2026-05-15"
- board text removed: "Factory-in-a-Box Control Unit v1.0"
