File: pcb_factory_control_unit/pcb_factory_control_unit.kicad_pcb (KiCad board)
At the start: 4 copper layers, 188 x 90 mm, 306 parts, among them J1 CAN, J10 WS2812_CH1, J11 WS2812_CH2, J12 LightBarrier1, J13 LightBarrier2, J14 PressureTransducer, J15 UEXT, J16 Malibotti, J17 Elevator, J18 Sorter, J19 Vacuum Pump, J2 STDC14, J20 Bus-Servo, J21 Cylinder Valve, J22 RoArm, J23 Conveyor, J24 Compressor, J25 Vacuum Valve, J26 Disturbance1, J27 Disturbance2, J28 INB, J29 Weight, J3 Micro_SD_Card_Det1, J4 DC IN, J5 USB STM32, J6 USB STM32, J7 I2C4, J8 I2C1B, J9 I2C1A, Q1 40N06D, Q2 BSS138, Q3 AO3400, Q4 AO3400, Q5 AO3400, Q6 AO3400, Q7 AO3400, Q8 AO3400, Q9 MMBT4403, SW1 Reset, SW2 Boot, U1 STM32H563VITx, U10 TMC2209, U11 74AHCT125, U12 HX711, U2 SIT3051TK, U3 LAN8742A, U4 TPS54202DDC, U5 TPS54202DDC, U6 MX26631DL, U7 AMS1117-3.3, U8 INA226, U9 TMC2209, X1 XL6009 (24V), Y1 25MHz, Y2 25MHz

Commit message: PCB WIP
Parts:
- moved R1 122.0 mm to (273.4, 98.1)
- moved C12 114.4 mm to (260.5, 89.1)
- moved C17 114.4 mm to (305.1, 95.4)
- moved L1 114.4 mm to (256.3, 92.0)
- moved R11 114.4 mm to (297.8, 101.3)
- moved R12 114.4 mm to (292.5, 99.0)
- moved R55 114.4 mm to (260.6, 86.6)
- moved C1 114.4 mm to (294.5, 101.5)
- moved C14 114.4 mm to (259.2, 89.2)
- moved C15 114.4 mm to (265.5, 72.9)
- moved C2 114.4 mm to (258.0, 89.0)
- moved C20 114.4 mm to (300.4, 72.5)
- moved C5 114.4 mm to (281.0, 96.2)
- moved NT1 114.4 mm to (256.3, 86.8)
- moved NT2 114.4 mm to (301.6, 72.6)
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Routing:
- net +3V3: track 648.3 -> 159.5 mm, vias 23 -> 9
- net +24V: track 359.9 -> 191.4 mm, vias 8 -> 2
- net I2C4_SCL: track 127.1 -> 0.00 mm, vias 3 -> 0
- net I2C4_SDA: track 120.1 -> 0.00 mm, vias 4 -> 0
- net I2C1_SCL: track 113.9 -> 0.00 mm, vias 3 -> 0
- net +5V: track 141.7 -> 27.9 mm, vias 1 -> 0
- net +12V: track 110.5 -> 0.00 mm, vias 2 -> 0
- net I2C1_SDA: track 108.3 -> 0.00 mm, vias 2 -> 0
- net INT_RGB: track 102.9 -> 0.00 mm, vias 1 -> 0
- net INT_TOF2: track 86.9 -> 0.00 mm, vias 1 -> 0
- net VALVE2: track 22.5 -> 109.1 mm
- net VALVE1: track 8.18 -> 89.9 mm
- net STEPPER_RX: track 80.5 -> 0.00 mm, vias 6 -> 0
- net I2C2_SCL: track 78.3 -> 0.00 mm, vias 3 -> 0
- net VALVE3: track 13.7 -> 89.0 mm, vias 2 -> 0
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
Commit message: WIP PCB
Parts:
- removed TP1: PE0, TestPoint:TestPoint_THTPad_D1.0mm_Drill0.5mm
- removed TP2: PD3, TestPoint:TestPoint_THTPad_D1.0mm_Drill0.5mm
- removed TP3: PA8, TestPoint:TestPoint_THTPad_D1.0mm_Drill0.5mm
- moved R71 155.3 mm to (122.9, 78.9), turned to 0 degrees
- moved J16 118.8 mm to (137.3, 138.7)
- moved SW2 118.2 mm to (183.4, 127.8), turned to 90 degrees
- moved J8 110.2 mm to (196.3, 138.8)
- moved J9 110.2 mm to (196.3, 145.0)
- moved J11 110.2 mm to (146.7, 138.7)
- moved SW1 102.1 mm to (189.1, 127.8), turned to 90 degrees
- moved C20 98.5 mm to (212.4, 116.6)
- moved C15 97.2 mm to (173.9, 105.5), turned to 180 degrees
- moved C69 86.8 mm to (235.2, 101.0)
- moved C100 74.4 mm to (261.2, 119.2)
- moved C73 74.4 mm to (260.9, 125.5)
- moved C74 74.4 mm to (279.3, 140.2)
- moved C79 74.4 mm to (268.0, 126.2)
- moved C81 74.4 mm to (269.8, 125.7)
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Connections:
- U1 pad 13: INT_TOF2 -> unconnected-(U1-PH1-Pad13)
- U1 pad 46: LED_INFO -> INT_TOF2
- U1 pad 57: VALVE1 -> VACUUM_VALVE
- U1 pad 63: LightBarrier1 -> VALVE2
- U1 pad 64: LightBarrier2 -> LightBarrier1
- U1 pad 65: unconnected-(U1-PC8-Pad65) -> LightBarrier2
- U1 pad 67: Net-(U1-PA8) -> VALVE1
- U1 pad 8: ETHERCAT_RESET -> unconnected-(U1-PC14-Pad8)
- U1 pad 84: Net-(U1-PD3) -> ETHERCAT_RESET
- U1 pad 86: VALVE2 -> unconnected-(U1-PD5-Pad86)
- U1 pad 97: Net-(U1-PE0) -> unconnected-(U1-PE0-Pad97)
Routing:
- net +24V: track 191.4 -> 41.2 mm
- net +3V3: track 159.5 -> 32.6 mm, vias 9 -> 2
- net SPI4_MISO: track 117.9 -> 29.5 mm
- net I2C4_SDA: track 0.00 -> 82.4 mm
- net I2C4_SCL: track 0.00 -> 76.5 mm
- net INT_TOF2: track 0.00 -> 76.3 mm, vias 0 -> 1
- net I2C2_SDA: track 0.00 -> 73.1 mm
- net VACUUM_VALVE: track 1.49 -> 74.1 mm, vias 0 -> 2
- net MALIBOTTI_RX: track 0.00 -> 71.7 mm, vias 0 -> 2
- net I2C2_SCL: track 0.00 -> 70.1 mm
- net MALIBOTTI_TX: track 0.00 -> 65.0 mm, vias 0 -> 2
- net unconnected-(J15-Pin_5-Pad5): track 60.3 -> 0.00 mm
- net ROBOT_TX: track 0.00 -> 59.9 mm, vias 0 -> 2
- net ROBOT_RX: track 0.00 -> 58.8 mm, vias 0 -> 2
- net LINKACTLED1: track 60.4 -> 2.21 mm
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Other:
- board size 188 x 90 mm -> 188 x 80 mm

Commit message: PCB WIP
Parts:
- moved R54 160.3 mm to (106.0, 134.1)
- moved C63 158.7 mm to (201.3, 133.1), turned to -90 degrees
- moved R55 158.2 mm to (108.6, 130.6)
- moved TP4 155.1 mm to (110.5, 129.8)
- moved C80 148.6 mm to (161.2, 102.2), turned to 0 degrees
- moved R81 141.6 mm to (154.6, 102.2)
- moved NT3 136.9 mm to (152.0, 92.7), turned to 0 degrees
- moved R11 135.2 mm to (165.9, 131.2), turned to 180 degrees
- moved C74 134.9 mm to (153.6, 91.2), turned to -135 degrees
- moved C17 131.7 mm to (179.6, 135.4), turned to 0 degrees
- moved Y2 131.2 mm to (154.8, 92.5), turned to 45 degrees
- moved C75 129.5 mm to (153.5, 94.0), turned to 135 degrees
- moved C10 128.8 mm to (171.6, 107.0), turned to 180 degrees
- moved C7 128.4 mm to (170.7, 121.7), turned to 180 degrees
- moved NT2 128.1 mm to (175.0, 91.8), turned to 0 degrees
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Connections:
- ETHERNET1 pad 8: GND -> GND1
- ETHERNET1 pad SH: GND -> GND1
- U1 pad 13: unconnected-(U1-PH1-Pad13) -> LED_INFO
- U1 pad 38: ROBOT_RX -> MALIBOTTI_RX
- U1 pad 39: ROBOT_TX -> MALIBOTTI_TX
- U1 pad 40: MALIBOTTI_RX -> ROBOT_RX
- U1 pad 41: MALIBOTTI_TX -> ROBOT_TX
- U11 pad 2: WS2812_1 -> WS2812_2
- U11 pad 3: WS2812_CH1 -> WS2812_CH2
- U11 pad 5: WS2812_2 -> WS2812_1
- U11 pad 6: WS2812_CH2 -> WS2812_CH1
Routing:
- net +3V3: track 32.6 -> 309.1 mm, vias 2 -> 21
- net +24V: track 41.2 -> 232.9 mm, vias 2 -> 7
- net +5V: track 16.8 -> 167.9 mm, vias 0 -> 4
- net CURRENT ALERT: track 0.00 -> 102.4 mm, vias 0 -> 2
- net STEPPER1_DIR: track 6.02 -> 101.7 mm, vias 1 -> 3
- net STEPPER2_DIR: track 0.00 -> 92.9 mm, vias 0 -> 2
- net STEPPER2_STEP: track 0.00 -> 91.0 mm, vias 0 -> 2
- net STEPPER_RX: track 0.00 -> 89.9 mm, vias 0 -> 2
- net STEPPER1_STEP: track 19.2 -> 95.6 mm, vias 1 -> 3
- net Net-(J19-Pin_3): track 0.00 -> 66.3 mm
- net HX711_SPI2_MISO: track 0.00 -> 52.6 mm
- net +12V: track 0.00 -> 52.5 mm, vias 0 -> 2
- net HX711_SPI2_MOSI: track 0.00 -> 51.5 mm
- net USB_VSENSE: track 0.00 -> 47.9 mm, vias 0 -> 2
- net PRESSURE_ADC: track 0.00 -> 45.0 mm, vias 0 -> 2
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
Commit message: wip
Parts:
- removed X1: XL6009 (24V), liebler_MODULES:DCDC-XL6009-boost
- added C102: 100uF, Capacitor_SMD:CP_Elec_6.3x7.7, F.Cu at (98.2, 90.1)
- added C103: 100uF, Capacitor_SMD:CP_Elec_6.3x7.7, F.Cu at (114.9, 115.3)
- added C104: 100uF, Capacitor_SMD:CP_Elec_6.3x7.7, F.Cu at (91.2, 89.8)
- added C105: 10u/35V, Capacitor_SMD:C_0805_2012Metric, F.Cu at (94.0, 98.1)
- added C106: 100uF, Capacitor_SMD:CP_Elec_6.3x7.7, F.Cu at (119.1, 108.2)
- added C107: 10u/35V, Capacitor_SMD:C_0805_2012Metric, F.Cu at (115.3, 121.9)
- added L12: 33uH, Inductor_SMD:L_Bourns_SRP1245A, F.Cu at (107.8, 103.5)
- added R106: 18k2, Resistor_SMD:R_0402_1005Metric, F.Cu at (110.7, 112.5)
- added R107: 1k, Resistor_SMD:R_0402_1005Metric, F.Cu at (88.3, 98.0)
- added U14: XL6009, Package_TO_SOT_SMD:TO-263-5_TabPin3, F.Cu at (94.8, 109.3)
- D2: value SMBJ24CA -> SS56C; footprint Diode_SMD:D_SMA -> Diode_SMD:D_SMC
- moved J14 76.3 mm to (183.4, 145.0)
- moved R47 71.2 mm to (185.8, 142.9), turned to -90 degrees
- moved R48 69.9 mm to (187.3, 142.4), turned to 180 degrees
- moved R30 46.7 mm to (131.1, 129.5), turned to 180 degrees
- moved D3 45.9 mm to (81.2, 129.9), turned to 180 degrees
- moved R33 44.9 mm to (131.1, 128.5), turned to 0 degrees
- moved C31 43.9 mm to (133.0, 129.8)
- moved C27 43.8 mm to (135.8, 123.9)
- moved C29 43.8 mm to (133.8, 123.9)
- moved C36 43.8 mm to (146.3, 124.6)
- moved C38 43.8 mm to (146.3, 130.6)
- moved U4 43.8 mm to (134.2, 127.6)
- moved C34 43.8 mm to (131.1, 127.5)
- moved L3 43.8 mm to (140.7, 127.6)
- moved R32 43.8 mm to (131.1, 126.5)
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Connections:
- C27 pad 2: +24V -> +20V
- C28 pad 2: +24V -> +20V
- C29 pad 2: +24V -> +20V
- C30 pad 2: +24V -> +20V
- C33 pad 2: Net-(D2-A2) -> Net-(D3-A2)
- D2 pad 1: GND -> +24V
- D2 pad 2: Net-(D2-A2) -> Net-(D2-A)
- J1 pad 1: CANH -> CANL
- J1 pad 3: CANL -> CANH
- J4 pad 1: Net-(D2-A2) -> Net-(D3-A2)
- Q1 pad 1: Net-(D2-A2) -> Net-(D3-A2)
- Q1 pad 2: Net-(D2-A2) -> Net-(D3-A2)
- Q1 pad 3: Net-(D2-A2) -> Net-(D3-A2)
- Q2 pad 2: Net-(D2-A2) -> Net-(D3-A2)
- R36 pad 2: Net-(D2-A2) -> Net-(D3-A2)
- R44 pad 2: +24V -> +20V
- U1 pad 38: MALIBOTTI_RX -> ROBOT_RX
- U1 pad 39: MALIBOTTI_TX -> ROBOT_TX
- U1 pad 40: ROBOT_RX -> MALIBOTTI_RX
- U1 pad 41: ROBOT_TX -> MALIBOTTI_TX
- U4 pad 3: +24V -> +20V
- U5 pad 3: +24V -> +20V
- U6 pad 5: Net-(D2-A2) -> Net-(D3-A2)
- U8 pad 9: +24V -> +20V
Routing:
- net +24V: track 232.9 -> 113.4 mm, vias 7 -> 0
- net STEPPER_EN: track 0.00 -> 101.2 mm, vias 0 -> 4
- net GND1: track 0.00 -> 76.6 mm
- net GND: track 22.3 -> 98.5 mm, vias 3 -> 33
- net +3V3: track 309.1 -> 237.8 mm, vias 21 -> 14
- net +5V: track 167.9 -> 106.2 mm, vias 4 -> 1
- net +20V: track 0.00 -> 51.9 mm
- net I2C4_SDA: track 83.7 -> 130.1 mm, vias 0 -> 3
- net I2C4_SCL: track 78.9 -> 123.9 mm, vias 0 -> 3
- net /EtherCAT/VDD33TXRX2: track 1.77 -> 41.7 mm, vias 0 -> 5
- net /EtherCAT/VDDCR: track 6.25 -> 42.1 mm, vias 0 -> 4
- net Net-(D2-A): track 0.00 -> 27.9 mm
- net Net-(D2-A2): track 25.8 -> 0.00 mm
- net STM32BOOT_TXD: track 0.00 -> 25.1 mm, vias 0 -> 3
- net /eth/LED1: track 0.00 -> 23.7 mm
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- added copper zone on B.Cu, net GNDA
- added copper zone on F.Cu, net GNDA
- added copper zone on In1.Cu, net GNDA
- added copper zone on In2.Cu, net GNDA
