File: pcb_factory_control_unit/pcb_factory_control_unit.kicad_sch (KiCad schematic)
At the start: 45 parts, among them J1 STDC14, J2 Micro_SD_Card_Det1, SW1 Reset, SW2 Boot, U1 STM32H563VITx, U10 SIT3051TK

Commit message: Changed LED ReverseMount Footprint, Removed PullUp, HSOS Logo
Parts:
- D1: footprint liebler_OPTO:LED_1206_3216Metric_ReverseMount -> LED_SMD:LED_1206_3216Metric_ReverseMount_Hole1.8x2.4mm

Commit message: Renaming & transfering test code
Other:
- note added: "ADC1 Input 18"
- note added: "CAN 1 Comunication"
- note added: "T15C1"
- note added: "T15C2"
- note added: "T2C1"
- note added: "T3C1"
- note added: "T4C3"
- note added: "T4C4"
- note added: "UART12"
- note added: "UART3"
- note added: "UART7"
- note removed: "CAN Comunication"
- note removed: "DEBUGGER"
