File: pcb_factory_control_unit/sensors.kicad_sch (KiCad schematic)
At the start: 17 parts, among them J23 Weight, J3 INB, Q4 MMBT4403, U9 HX711

Commit message: Control Unit PCB: schematic rework (PSU, MX26631DL, XL6009 module, ERC fixes), new placement on 90 mm high board
Parts:
- Q9: renamed from Q4; footprint liebler_SEMICONDUCTORS:SOT-23_smaller -> Package_TO_SOT_SMD:SOT-23
- renumbered C54 to C66, C55 to C67, C56 to C68, C60 to C69, C57 to C70, C59 to C71, J3 to J28, J23 to J29, L4 to L6, L6 to L7, R57 to R76, R58 to R77, R59 to R78, R60 to R79, R61 to R80, U9 to U12
