File: pcb_factory_control_unit/conn.kicad_sch (KiCad schematic)
At the start: 21 parts, among them J6 USB STM32

Commit message: PCB Control Unit: add EEPROM-select jumpers on EtherCAT ESC, new J7 connector
ethercat_esc.kicad_sch: add EESDA solder jumpers JP4/JP5 with pull-up
resistor R89 (3k3) and a RUNLED_PU label, wired to GND/+3V3.
conn.kicad_sch: add 4-pin connector J7 (+12V/GND).
Parts:
- added J7: Conn_01x04, symbol Connector_Generic:Conn_01x04
- added J?: Vacuum Pump, liebler_CONN:JST_XH_B3B-XH-A_1x03_P2.50mm_Vertical_smaller, symbol Connector_Generic:Conn_01x03
- renumbered LB2 to J?, LB3 to J?, LB1 to J?
Connections:
- net GND: now also J?.2 (Pin_2)
- new net +12V: J?.1 (Pin_1)
- new net VACUUM_PUMP_PWM: J?.3 (Pin_3)

Commit message: Control Unit PCB: schematic rework (PSU, MX26631DL, XL6009 module, ERC fixes), new placement on 90 mm high board
Parts:
- removed CanBus1: CAN, liebler_CONN:JST_XH_B3B-XH-A_1x03_P2.50mm_Vertical_smaller, symbol Connector_Generic:Conn_01x03
- removed J7: Conn_01x04, symbol Connector_Generic:Conn_01x04
- removed J?: Vacuum Pump, liebler_CONN:JST_XH_B3B-XH-A_1x03_P2.50mm_Vertical_smaller, symbol Connector_Generic:Conn_01x03
- removed J?: LightBarrier3, liebler_CONN:JST_XH_B3B-XH-A_1x03_P2.50mm_Vertical_smaller, symbol Connector_Generic:Conn_01x03
- removed JP1, JP2, JP3: 5-24, Jumper:SolderJumper-3_P1.3mm_Open_RoundedPad1.0x1.5mm_NumberLabels, symbol Jumper:SolderJumper_3_Open
- removed UEXT1: BH10S, ayluna:UEXTM-PTH, symbol agua:BH10S
- added J15: UEXT, Connector_IDC:IDC-Header_2x05_P2.54mm_Vertical, symbol Connector_Generic:Conn_02x05_Odd_Even
- IJ1: renamed from I2C2; value TOF2 -> I2C2
- J7: renamed from I2C4; value TOF3 -> I2C4
- J8: renamed from I2C1B1; value TOF1 -> I2C1B
- J9: renamed from I2C1A1; value RGB -> I2C1A
- gave numbers to parts that had none: 2
- renumbered Leds1 to J10, Leds2 to J11, Pressure1 to J14, Malibotti1 to J16, R35 to R45, R36 to R46, R37 to R47, R38 to R48
Connections:
- net +24V: now also J12.1 (Pin_1), J13.1 (Pin_1)
- net +3V3: now also J15.1 (Pin_1)
- net GND: now also J6.SH (SHIELD), J15.2 (Pin_2); no longer J6.S1 (SHIELD)
- net SPI4_CLK: now also J15.9 (Pin_9)
- net SPI4_MISO: now also J15.7 (Pin_7)
- net SPI4_MOSI: now also J15.8 (Pin_8)
- no-connect marks 2 -> 7
Other:
- note added: "I2C"
- note added: "Light Barriers"
- note added: "Malibotti"
- note added: "RGB-LEDs"
- note added: "UEXT"
- note removed: "Connectors"
- note removed: "LEDS"
- moved on the sheet: IJ1, J10, J11, J12, J13, J14, J16, J7, J8, J9, R47, R48

Commit message: FCB ready for review
Parts:
- J14: value PressureTransducer -> PressureSns
Other:
- note added: "Pressure"
Changed lines of the file:
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@@
 		)
 	)
-	(text "RGB-LEDs"
+	(text "Pressure"
 		(exclude_from_sim no)
 		(at 58.42 123.19 0)
@@
 			)
 		)
-		(property "Value" "PressureTransducer"
+		(property "Value" "PressureSns"
 			(at 90.17 124.46 90)
 			(show_name no)
