File: pcb_factory_control_unit/psu.kicad_sch (KiCad schematic)
At the start: 32 parts, among them J4 DC IN, J5 USB STM32, U12 TPS54202DDC, U4 TPS54202DDC, U5 AMS1117-3.3, U6 INA226, X1 MT3608

Commit message: Changed LED ReverseMount Footprint, Removed PullUp, HSOS Logo
Parts:
- removed R89: 10k, Resistor_SMD:R_0402_1005Metric, symbol Device:R
Other:
- note added: "Activate Pullup in STM32!"

Commit message: Control Unit PCB: schematic rework (PSU, MX26631DL, XL6009 module, ERC fixes), new placement on 90 mm high board
Parts:
- added C33: 1u/50V, Capacitor_SMD:C_0805_2012Metric, symbol Device:C
- added C41: u1/16V, Capacitor_SMD:C_0402_1005Metric, symbol Device:C
- added C42, C44: 10u/50V, Capacitor_SMD:C_1210_3225Metric, symbol Device:C
- added C45: 100u/50V, Capacitor_SMD:CP_Elec_8x10, symbol Device:C_Polarized
- added D2: SMBJ24CA, Diode_SMD:D_SMA, symbol Diode:SMAJ22CA
- added D3: SMAJ22CA, Diode_SMD:D_SMA, symbol Diode:SMAJ22CA
- added L5: 4.7uH, Inductor_SMD:L_Bourns_SRP1245A, symbol Device:L
- added Q1: 40N06D, Package_SON:VSON-8_3.3x3.3mm_P0.65mm_NexFET, symbol Transistor_FET:CSD18543Q3A
- added Q2: BSS138, Package_TO_SOT_SMD:SOT-23, symbol Transistor_FET:BSS138
- added R36, R40: 330k, Resistor_SMD:R_0402_1005Metric, symbol Device:R
- added R37: 6k8, Resistor_SMD:R_0402_1005Metric, symbol Device:R
- added R38: 15k, Resistor_SMD:R_0402_1005Metric, symbol Device:R
- added R39: 1k, Resistor_SMD:R_0402_1005Metric, symbol Device:R
- added R41: 22k, Resistor_SMD:R_0402_1005Metric, symbol Device:R
- added R42, R43: 10k, Resistor_SMD:R_0402_1005Metric, symbol Device:R
- added U6: MX26631DL, Package_DFN_QFN:Texas_RGE0024H_VQFN-24-1EP_4x4mm_P0.5mm_EP2.7x2.7mm_ThermalVias, symbol Power_Management:TPS26631RGE
- U4: footprint Package_TO_SOT_SMD:SOT-23-6_Handsoldering -> Package_TO_SOT_SMD:SOT-23-6
- U5: renamed from U12; footprint Package_TO_SOT_SMD:SOT-23-6_Handsoldering -> Package_TO_SOT_SMD:SOT-23-6
- X1: value MT3608 -> XL6009 (24V); footprint liebler_MODULES:DCDC_MT3608 -> liebler_MODULES:DCDC-XL6009-boost
- renumbered C76 to C28, C28 to C29, C80 to C30, C29 to C31, C84 to C32, C30 to C34, C88 to C35, C31 to C36, C89 to C37, C32 to C38, C98 to C39, C33 to C40, C34 to C43, C35 to C46, L10 to L4, R31 to R30, R87 to R31, R88 to R34, R96 to R35, R34 to R44, U5 to U7, U6 to U8
Connections:
- net +24V: now also C27.2, C28.2, C29.2, C30.2, R44.2, U4.3 (VIN), U5.3 (VIN), U8.9 (Vin-); no longer X1.4 (out+)
- net +VDC: now also C44.1, C45.1, L5.2; no longer J4.1, J5.A4 (VBUS), J5.A9 (VBUS), J5.B4 (VBUS), J5.B9 (VBUS)
- net GND: now also J5.SH (SHIELD), C33.1, C41.1, C42.2, C44.2, C45.2, D2.1 (A1), D3.1 (A1), R39.2, R41.2, R42.1, R43.1, U6.11 (MODE), U6.25 (GND), U6.8 (GND); no longer J5.S1 (SHIELD)
- removed net 5-24V: C27.2, C28.2, C29.2, C30.2, R44.2, U4.3 (VIN), U5.3 (VIN), U8.9 (Vin-), X1.1 (In+)
- new net: R42.2, U6.10 (ILIM)
- new net: R40.1, R41.1, U6.15 (PGTH)
- new net: D3.2 (A2), J5.A4 (VBUS), J5.A9 (VBUS), J5.B4 (VBUS), J5.B9 (VBUS), X1.1 (In+)
- new net: C33.2, D2.2 (A2), J4.1, Q1.1 (S), Q1.2 (S), Q1.3 (S), Q2.2 (S), R36.2, U6.5 (IN_SYS), X1.4 (out+)
- new net: C42.1, L5.1, R40.2, U6.17 (OUT), U6.18 (OUT)
- new net: R38.1, R39.1
- new net: R37.1, R38.2, U6.7 (OVP)
- new net: Q2.1 (G), U6.4 (DRV)
- new net: Q1.4 (G), Q2.3 (D), U6.3 (B_GATE)
- new net: R43.2, U6.13 (IMON)
- new net: Q1.5 (D), U6.1 (IN), U6.2 (IN)
- new net: R36.1, R37.2, U6.6 (UVLO)
- new net: C41.2, U6.9 (dVdT)
- no-connect marks 8 -> 11
Other:
- note added: "PSU Eingang: USB-PD 20V → XL6009 (24V) ODER DC-Buchse 24V (nie beide gleichzeitig anschließen!) → MX26631 → Pi-Filter → +VDC"
- note added: "Pi-Filter"
- note added: "U5 = MX26631DL (Wuxi Maxinmicro, LCSC C18197523), pinkompatibel zu TI TPS26631RGE. Abweichungen zum TI-Original: - ILIM: I_lim ≈ 38 / R39[kΩ] (TI: 18 / R), R 5…100 kΩ, max. 5 A → R39 = 10k ≈ 3,8 A (mit TI-Chip wäre 5k1 richtig) - Überstrompuls 1,5 × I_lim (TI: 2 × I_lim für ca. 25 ms) - Schwellen UVLO/OVP 1,21 V, PGTH 1,24 V (TI: 1,20 V) → UVLO ≈ 18,7 V, OVP ≈ 26,7 V, PGOOD ≈ 19,8 V - Betriebsspa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"
- note added: "XL6009-Modul auf 24,0V trimmen"
- note removed: "24V - 5-24V"
- note removed: "Barrel Jack 24V"
- note removed: "USB PD"
- moved on the sheet: C27, C29, C31, C34, C36, C38, C40, C43, J4, J5, L3, R30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

Commit message: wip
Parts:
- removed D2: SMBJ24CA, Diode_SMD:D_SMA, symbol Diode:SMAJ22CA
- removed X1: XL6009 (24V), liebler_MODULES:DCDC-XL6009-boost, symbol liebler_MODULES:XL_4015
- added C102, C103, C104, C106: 100uF, Capacitor_SMD:CP_Elec_6.3x7.7, symbol Device:C_Polarized
- added C105, C107: 10u/35V, Capacitor_SMD:C_0805_2012Metric, symbol Device:C
- added D2: SS56C, Diode_SMD:D_SMC, symbol Device:D_Schottky
- added L12: 33uH, Inductor_SMD:L_Bourns_SRP1245A, symbol Device:L
- added R106: 18k2, Resistor_SMD:R_0402_1005Metric, symbol Device:R
- added R107: 1k, Resistor_SMD:R_0402_1005Metric, symbol Device:R
- added U14: XL6009, Package_TO_SOT_SMD:TO-263-5_TabPin3, symbol liebler_SEMICONDUCTORS:XL6009
Connections:
- net +24V: now also C103.1, C106.1, C107.2, D2.1 (K), R106.1; no longer C27.2, C28.2, C29.2, C30.2, R44.2, U4.3 (VIN), U5.3 (VIN), U8.9 (Vin-)
- net GND: now also C102.2, C103.2, C104.2, C105.1, C106.2, C107.1, R107.1, U14.1 (GND)
- net at D3.2 (A2), J5.A4 (VBUS), J5.A9 (VBUS)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: now also C33.2, J4.1, Q1.1 (S), Q1.2 (S), Q1.3 (S), Q2.2 (S), R36.2, U6.5 (IN_SYS)
- new net: D2.2 (A), L12.1, U14.3 (SW)
- new net: R106.2, R107.2, U14.5 (FB)
- new net +20V: C102.1, C104.1, C105.2, C27.2, C28.2, C29.2, C30.2, L12.2, R44.2, U14.4 (VIN), U4.3 (VIN), U5.3 (VIN), U8.9 (Vin-)
- no-connect marks 11 -> 12
Other:
- note removed: "XL6009-Modul auf 24,0V trimmen"
- moved on the sheet: D3

Commit message: New Step Up Controller
Parts:
- removed C102, C103, C104, C106: 100uF, Capacitor_SMD:CP_Elec_6.3x7.7, symbol Device:C_Polarized
- removed C107: 10u/35V, Capacitor_SMD:C_0805_2012Metric, symbol Device:C
- removed U14: XL6009, Package_TO_SOT_SMD:TO-263-5_TabPin3, symbol liebler_SEMICONDUCTORS:XL6009
- added C102, C103, C104: 10u/50, Capacitor_SMD:C_1210_3225Metric, symbol Device:C
- added C108, C109: 47n, Capacitor_SMD:C_0805_2012Metric, symbol Device:C
- added C110, C111: 4u7/35, Capacitor_SMD:C_0805_2012Metric, symbol Device:C
- added C112: 1n5, Capacitor_SMD:C_0805_2012Metric, symbol Device:C
- added R108: 1k, Resistor_SMD:R_0402_1005Metric, symbol Device:R
- added R109, R110: 82k, Resistor_SMD:R_0402_1005Metric, symbol Device:R
- added U15: TPS55340, Package_DFN_QFN:WQFN-16-1EP_3x3mm_P0.5mm_EP1.68x1.68mm_ThermalVias, symbol liebler_SEMICONDUCTORS:TPS55340
- C105: value 10u/35V -> u1/35
- L12: value 33uH -> 10uH; footprint Inductor_SMD:L_Bourns_SRP1245A -> Inductor_SMD:L_Abracon_ASPI-0630LR; LCSC (none) -> C475521; MPN (none) -> FXL0650-100-M
- R106: value 18k2 -> M1
- R107: value 1k -> 10k
Connections:
- net +20V: now also C110.2, C111.2, U15.2 (VIN), U15.3 (EN)
- net +24V: now also C102.1, C103.1, C104.1, R110.1; no longer R106.1
- net GND: now also C102.2, C103.2, C104.2, C108.1, C109.1, C110.1, C111.1, C112.1, R109.1, U15.10 (NC), U15.11 (PGND), U15.12 (PGND), U15.13 (PGND), U15.14 (NC), U15.17 (AGND), U15.5 (SYNC), U15.6 (AGND); no longer U6.11 (MODE), U6.25 (GND), U6.8 (GND)
- net at R42.2: no longer U6.10 (ILIM)
- net at R40.1, R41.1: no longer U6.15 (PGTH)
- net at C33.2, D3.2 (A2), J4.1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: no longer U6.5 (IN_SYS)
- net at D2.2 (A), L12.1: now also U15.1 (SW), U15.15 (SW), U15.16 (SW)
- net at R37.1, R38.2: no longer U6.7 (OVP)
- net at Q2.1 (G): no longer U6.4 (DRV)
- net at Q1.4 (G), Q2.3 (D): no longer U6.3 (B_GATE)
- net at R106.2, R107.2: now also U15.8 (FB)
- net at R43.2: now also U6.9 (dVdT); no longer U6.13 (IMON)
- net at U6.12 (~{SHDN}): now also R36.1, R37.2
- net at C41.2: no longer U6.9 (dVdT)
- new net: C108.2, R108.2
- new net: R106.1, R110.2
- new net: C112.2, R108.1, U15.7 (COMP)
- new net: R109.2, U15.9 (FREQ)
- new net: C109.2, U15.4 (SS)
- new net: U6.25 (GND), U6.8 (GND)
- now unconnected: U6.6 (UVLO)
- no-connect marks 12 -> 11
Other:
- note added: "PSU Eingang: USB-PD (20V) ODER DC-Buchse 24V (nie beide gleichzeitig anschließen!) → MX26631 → Pi-Filter → +VDC"
- note removed: "PSU Eingang: USB-PD 20V → XL6009 (24V) ODER DC-Buchse 24V (nie beide gleichzeitig anschließen!) → MX26631 → Pi-Filter → +VDC"
- note removed: "Pi-Filter"
- moved on the sheet: C105, D2, L12, R106, R107, U6

Commit message: Step Up Converter
Parts:
- C108, C109, C112: footprint Capacitor_SMD:C_0805_2012Metric -> Capacitor_SMD:C_0402_1005Metric
Changed lines of the file:
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@@
 			)
 		)
-		(property "Footprint" "Capacitor_SMD:C_0805_2012Metric"
+		(property "Footprint" "Capacitor_SMD:C_0402_1005Metric"
 			(at 160.3248 148.59 0)
 			(hide yes)
@@
 			)
 		)
-		(property "Footprint" "Capacitor_SMD:C_0805_2012Metric"
+		(property "Footprint" "Capacitor_SMD:C_0402_1005Metric"
 			(at 167.9448 148.59 0)
 			(hide yes)
@@
 			)
 		)
-		(property "Footprint" "Capacitor_SMD:C_0805_2012Metric"
+		(property "Footprint" "Capacitor_SMD:C_0402_1005Metric"
 			(at 181.9148 148.59 0)
 			(hide yes)

Commit message: WIP
Parts:
- removed U6: MX26631DL, Package_DFN_QFN:Texas_RGE0024H_VQFN-24-1EP_4x4mm_P0.5mm_EP2.7x2.7mm_ThermalVias, symbol Power_Management:TPS26631RGE
- added U14: TPS26631RGE, Package_DFN_QFN:Texas_RGE0024H_VQFN-24-1EP_4x4mm_P0.5mm_EP2.7x2.7mm_ThermalVias, symbol liebler_SEMICONDUCTORS:TPS26631RGE
Connections:
- net GND: now also U14.11 (MODE), U14.25 (GND), U14.8 (GND)
- net at R42.2: now also U14.10 (ILIM)
- net at R40.1, R41.1: now also U14.15 (PGTH)
- net DC_IN: now reaches C33.2, D3.2 (A2), J4.1, J5.A4 (VBUS), J5.A9 (VBUS), J5.B4 (VBUS), J5.B9 (VBUS), Q1.1 (S), Q1.2 (S), Q1.3 (S), Q2.2 (S), R36.2
- net DC_IN: now also U14.5 (IN_SYS)
- net DC_OUT: now reaches C42.1, L5.1, R40.2
- net DC_OUT: now also U14.17 (OUT), U14.18 (OUT)
- net at R37.1, R38.2: now also U14.7 (OVP)
- net at Q2.1 (G): now also U14.4 (DRV)
- net at Q1.4 (G), Q2.3 (D): now also U14.3 (B_GATE)
- net at R43.2: now also U14.13 (IMON)
- net FUSE_IN: now reaches Q1.5 (D)
- net FUSE_IN: now also U14.1 (IN), U14.2 (IN)
- net at R36.1, R37.2: now also U14.6 (UVLO)
- net at C41.2: now also U14.9 (dVdT)
Other:
- moved on the sheet: R40

Commit message: FCB ready for review
Connections:
- net STEPUP_SW: now reaches D2.2 (A), L12.1, U15.1 (SW), U15.15 (SW), U15.16 (SW)
Changed lines of the file:
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@@
+		)
+	)
+	(label "STEPUP_SW"
+		(at 204.47 120.65 0)
+		(effects
+			(font
+				(size 1.27 1.27)
+			)
+			(justify left bottom)
 		)
 	)
